Commit message: Building robot_stage1 with variables and more parts

File: models/robots/robot_stage1.xacro (robot description, xacro)
@@ -1,74 +1,156 @@
 <?xml version="1.0"?>
 <robot xmlns:xacro="http://www.ros.org/wiki/xacro" name="myrobot">
+  <!-- Body properties -->
   <xacro:property name="body_radius" value="0.2" />
   <xacro:property name="body_length" value="0.6" />
-  <xacro:property name="leg_radius" value="0.1" />
-  <xacro:property name="leg_length" value="0.4" />
-  <xacro:property name="leg_offset" value="0.25" />
+  <xacro:property name="body_mass" value="2" />
+  <xacro:property name="body_ixx" value="0.4" />
+  <xacro:property name="body_iyy" value="0.4" />
+  <xacro:property name="body_izz" value="0.2" />
+  <!-- Thigh properties -->
+  <xacro:property name="thigh_radius" value="0.1" />
+  <xacro:property name="thigh_length" value="0.25" />
+  <xacro:property name="thigh_mass" value="2" />
+  <xacro:property name="thigh_ixx" value="0.02" />
+  <xacro:property name="thigh_iyy" value="0.02" />
+  <xacro:property name="thigh_izz" value="0.01" />
+  <!-- Shin properties -->
+  <xacro:property name="shin_radius" value="0.08" />
+  <xacro:property name="shin_length" value="0.2" />
+  <xacro:property name="shin_mass" value="1.5" />
+  <xacro:property name="shin_ixx" value="0.015" />
+  <xacro:property name="shin_iyy" value="0.015" />
+  <xacro:property name="shin_izz" value="0.008" />
+  <!-- Foot properties -->
+  <xacro:property name="foot_length" value="0.3" />
+  <xacro:property name="foot_width" value="0.2" />
+  <xacro:property name="foot_height" value="0.05" />
+  <xacro:property name="foot_mass" value="0.5" />
+  <xacro:property name="foot_ixx" value="0.002" />
+  <xacro:property name="foot_iyy" value="0.002" />
+  <xacro:property name="foot_izz" value="0.001" />
+  <xacro:property name="leg_offset" value="0.0" />
+  <!-- Head properties -->
   <xacro:property name="head_radius" value="0.15" />
+  <xacro:property name="head_mass" value="0.1" />
+  <xacro:property name="head_ixx" value="0.01" />
+  <xacro:property name="head_iyy" value="0.01" />
+  <xacro:property name="head_izz" value="0.01" />
+  <!-- IMU properties -->
+  <xacro:property name="imu_length" value="0.03" />
+  <xacro:property name="imu_width" value="0.05" />
+  <xacro:property name="imu_height" value="0.05" />
+  <xacro:property name="imu_mass" value="0.01" />
+  <xacro:property name="imu_ixx" value="0.0001" />
+  <xacro:property name="imu_iyy" value="0.0001" />
+  <xacro:property name="imu_izz" value="0.0001" />
+  <!-- Materials -->
   <material name="robot_material">
     <color rgba="0.37 0.09 0.09 1"/>
   </material>
+  <!-- Body (main cylinder) -->
   <link name="base_link">
+  <origin xyz="0 0 0"/>
     <visual>
+      <origin xyz="0 0 ${body_length/2 + thigh_length}"/>
       <geometry>
         <cylinder length="${body_length}" radius="${body_radius}"/>
       </geometry>
-	  <material name="robot_material"/>
+      <material name="robot_material"/>
     </visual>
-	<collision>
+    <collision>
+      <origin xyz="0 0 ${body_length/2 + thigh_length}"/>
       <geometry>
         <cylinder length="${body_length}" radius="${body_radius}"/>
       </geometry>
     </collision>
-	<inertial>
-      <mass value="10"/>
-      <inertia ixx="0.4" ixy="0.0" ixz="0.0" iyy="0.4" iyz="0.0" izz="0.2"/>
+    <inertial>
+      <mass value="${body_mass}"/>
+      <inertia ixx="${body_ixx}" ixy="0.0" ixz="0.0" iyy="${body_iyy}" iyz="0.0" izz="${body_izz}"/>
     </inertial>
   </link>
-  <xacro:macro name="leg" params="prefix reflect">
-	  <link name="${prefix}_leg_link">
-		<visual>
-		  <geometry>
-			<cylinder length="${leg_length}" radius="${leg_radius}"/>
-		  </geometry>
-		  <origin rpy="0 0 0" xyz="0 0 -${leg_length/2}"/>
-		  <material name="robot_material"/>
-		</visual>
-		<collision>
-		  <geometry>
-			<cylinder length="${leg_length}" radius="${leg_radius}"/>
-		  </geometry>
-		  <origin rpy="0 0 0" xyz="0 0 -${leg_length/2}"/>
-		</collision>
-	  </link>
-	  <joint name="base_to_${prefix}_leg" type="continuous">
-		<parent link="base_link"/>
-		<child link="${prefix}_leg_link"/>
-		<origin xyz="0 ${leg_offset*reflect} -${body_length/2}"/>
-		<axis xyz="0 1 0"/>
-	  </joint>
-  </xacro:macro>
-  <xacro:leg prefix="right" reflect="-1" />
-  <xacro:leg prefix="left" reflect="1" />
+  <!-- IMU (simulated sensor, offset from body center) -->
+  <link name="imu_link">
+    <visual>
+      <geometry>
+        <box size="${imu_length} ${imu_width} ${imu_height}"/>
+      </geometry>
+      <origin xyz="0 0 0" rpy="0 0 0"/>
+      <material name="robot_material"/>
+    </visual>
+    <collision>
+      <geometry>
+        <box size="${imu_length} ${imu_width} ${imu_height}"/>
+      </geometry>
+      <origin xyz="0 0 0" rpy="0 0 0"/>
+    </collision>
+    <inertial>
+      <mass value="${imu_mass}"/>
+      <inertia ixx="${imu_ixx}" ixy="0.0" ixz="0.0" iyy="${imu_iyy}" iyz="0.0" izz="${imu_izz}"/>
+    </inertial>
+  </link>
+  <joint name="base_to_imu" type="fixed">
+    <parent link="base_link"/>
+    <child link="imu_link"/>
+    <origin xyz="${body_radius + imu_length/2} 0 ${imu_height/2 + thigh_length + body_length/3}" rpy="0 0 0"/>
+  </joint>
+  <!-- Head (sphere) -->
   <link name="head_link">
     <visual>
+      <origin rpy="0 0 0" xyz="0 0 ${head_radius + thigh_length}"/>
       <geometry>
         <sphere radius="${head_radius}"/>
       </geometry>
-	  <origin rpy="0 0 0" xyz="0 0 ${head_radius}"/>
       <material name="robot_material"/>
     </visual>
-	<collision>
+    <collision>
+      <origin rpy="0 0 0" xyz="0 0 ${head_radius + thigh_length}"/>
       <geometry>
         <sphere radius="${head_radius}"/>
       </geometry>
-	  <origin rpy="0 0 0" xyz="0 0 ${head_radius}"/>
     </collision>
+    <inertial>
+      <mass value="${head_mass}"/>
+      <inertia ixx="${head_ixx}" ixy="0.0" ixz="0.0" iyy="${head_iyy}" iyz="0.0" izz="${head_izz}"/>
+    </inertial>
   </link>
+  <!-- Leg macro (creates left/right leg: thigh, shin, foot) -->
+  <xacro:macro name="leg" params="prefix reflect">
+    <!-- Thigh -->
+    <link name="${prefix}_thigh_link">
+      <visual>
+        <geometry>
+          <cylinder length="${thigh_length}" radius="${thigh_radius}"/>
+        </geometry>
+        <origin rpy="0 0 0" xyz="0 0 -${thigh_length/2}"/>
+        <material name="robot_material"/>
+      </visual>
+      <collision>
+        <geometry>
+          <cylinder length="${thigh_length}" radius="${thigh_radius}"/>
+        </geometry>
+        <origin rpy="0 0 0" xyz="0 0 -${thigh_length/2}"/>
+      </collision>
+      <inertial>
+        <mass value="${thigh_mass}"/>
+        <inertia ixx="${thigh_ixx}" ixy="0.0" ixz="0.0" iyy="${thigh_iyy}" iyz="0.0" izz="${thigh_izz}"/>
+      </inertial>
+    </link>
+    <!-- Hip joint: base_link to thigh -->
+    <joint name="base_to_${prefix}_thigh" type="revolute">
+      <parent link="base_link"/>
+      <child link="${prefix}_thigh_link"/>
+      <origin xyz="0 ${(body_radius + thigh_radius + leg_offset) * reflect} ${thigh_length}"/>
+      <axis xyz="0 1 0"/>
+      <limit lower="-1.57" upper="1.57" effort="50" velocity="5"/>
+    </joint>
+  </xacro:macro>
+  <!-- Instantiate right and left legs -->
+  <xacro:leg prefix="right" reflect="-1" />
+  <xacro:leg prefix="left" reflect="1" />
   <joint name="base_to_head" type="fixed">
     <parent link="base_link"/>
     <child link="head_link"/>
-	<origin xyz="0 0 ${body_length/2}"/>
+	<origin xyz="0 0 ${body_length}"/>
   </joint>
 </robot>

Commit message: Adding legs to the robot_stage1

File: models/robots/robot_stage1.xacro (robot description, xacro)
@@ -16,5 +16,5 @@
   <xacro:property name="thigh_izz" value="0.01" />
   <!-- Shin properties -->
-  <xacro:property name="shin_radius" value="0.08" />
+  <xacro:property name="shin_radius" value="0.05" />
   <xacro:property name="shin_length" value="0.2" />
   <xacro:property name="shin_mass" value="1.5" />
@@ -51,7 +51,9 @@
   <!-- Body (main cylinder) -->
   <link name="base_link">
-  <origin xyz="0 0 0"/>
+    <origin xyz="0 0 0"/>
     <visual>
-      <origin xyz="0 0 ${body_length/2 + thigh_length}"/>
+      <!-- body_length/2 shifts the Z plane from the cylinder's center to its base -->
+      <!-- thigh_length + shin_length gives space for the legs -->
+      <origin xyz="0 0 ${body_length/2 + thigh_length + shin_length}"/>
       <geometry>
         <cylinder length="${body_length}" radius="${body_radius}"/>
@@ -60,5 +62,5 @@
     </visual>
     <collision>
-      <origin xyz="0 0 ${body_length/2 + thigh_length}"/>
+      <origin xyz="0 0 ${body_length/2 + thigh_length + shin_length}"/>
       <geometry>
         <cylinder length="${body_length}" radius="${body_radius}"/>
@@ -73,15 +75,15 @@
   <link name="imu_link">
     <visual>
+      <origin xyz="0 0 0" rpy="0 0 0"/>
       <geometry>
         <box size="${imu_length} ${imu_width} ${imu_height}"/>
       </geometry>
-      <origin xyz="0 0 0" rpy="0 0 0"/>
       <material name="robot_material"/>
     </visual>
     <collision>
+      <origin xyz="0 0 0" rpy="0 0 0"/>
       <geometry>
         <box size="${imu_length} ${imu_width} ${imu_height}"/>
       </geometry>
-      <origin xyz="0 0 0" rpy="0 0 0"/>
     </collision>
     <inertial>
@@ -93,10 +95,15 @@
     <parent link="base_link"/>
     <child link="imu_link"/>
-    <origin xyz="${body_radius + imu_length/2} 0 ${imu_height/2 + thigh_length + body_length/3}" rpy="0 0 0"/>
+    <!-- Since the body is positioned at 0 0 0, move the joint considering the length of the legs and part of the body -->
+    <!-- Z: Move the IMU shin_length + thigh_length, to place it above the legs -->
+    <!-- Z: Move the IMU body_length/3 to place it around the middle of the body -->
+    <!-- X: Move the IMU body_radius to place it at the edge of the body -->
+    <origin xyz="${body_radius} 0 ${shin_length + thigh_length + body_length/3 }" rpy="0 0 0"/>
   </joint>
   <!-- Head (sphere) -->
   <link name="head_link">
     <visual>
-      <origin rpy="0 0 0" xyz="0 0 ${head_radius + thigh_length}"/>
+      <!-- head_radius shifts the Z plane from the heads's center to its base -->
+      <origin rpy="0 0 0" xyz="0 0 ${head_radius}"/>
       <geometry>
         <sphere radius="${head_radius}"/>
@@ -105,5 +112,5 @@
     </visual>
     <collision>
-      <origin rpy="0 0 0" xyz="0 0 ${head_radius + thigh_length}"/>
+      <origin rpy="0 0 0" xyz="0 0 ${head_radius}"/>
       <geometry>
         <sphere radius="${head_radius}"/>
@@ -115,4 +122,10 @@
     </inertial>
   </link>
+  <joint name="base_to_head" type="fixed">
+    <parent link="base_link"/>
+    <child link="head_link"/>
+    <!-- Since the body is positioned at 0 0 0, move the joint up considering the length of the legs and the body -->
+	  <origin xyz="0 0 ${shin_length + thigh_length + body_length}"/>
+  </joint>
   <!-- Leg macro (creates left/right leg: thigh, shin, foot) -->
   <xacro:macro name="leg" params="prefix reflect">
@@ -120,15 +133,15 @@
     <link name="${prefix}_thigh_link">
       <visual>
+        <origin rpy="0 0 0" xyz="0 0 -${thigh_length/2}"/>
         <geometry>
           <cylinder length="${thigh_length}" radius="${thigh_radius}"/>
         </geometry>
-        <origin rpy="0 0 0" xyz="0 0 -${thigh_length/2}"/>
         <material name="robot_material"/>
       </visual>
       <collision>
+        <origin rpy="0 0 0" xyz="0 0 -${thigh_length/2}"/>
         <geometry>
           <cylinder length="${thigh_length}" radius="${thigh_radius}"/>
         </geometry>
-        <origin rpy="0 0 0" xyz="0 0 -${thigh_length/2}"/>
       </collision>
       <inertial>
@@ -141,7 +154,35 @@
       <parent link="base_link"/>
       <child link="${prefix}_thigh_link"/>
-      <origin xyz="0 ${(body_radius + thigh_radius + leg_offset) * reflect} ${thigh_length}"/>
+      <origin xyz="0 ${(body_radius + thigh_radius + leg_offset) * reflect} ${thigh_length + shin_length}"/>
       <axis xyz="0 1 0"/>
       <limit lower="-1.57" upper="1.57" effort="50" velocity="5"/>
+    </joint>
+    <!-- Shin -->
+    <link name="${prefix}_shin_link">
+      <visual>
+        <origin rpy="0 0 0" xyz="0 0 -${shin_length/2}"/>
+        <geometry>
+          <cylinder length="${shin_length}" radius="${shin_radius}"/>
+        </geometry>
+        <material name="robot_material"/>
+      </visual>
+      <collision>
+        <origin rpy="0 0 0" xyz="0 0 -${shin_length/2}"/>
+        <geometry>
+          <cylinder length="${shin_length}" radius="${shin_radius}"/>
+        </geometry>
+      </collision>
+      <inertial>
+        <mass value="${shin_mass}"/>
+        <inertia ixx="${shin_ixx}" ixy="0.0" ixz="0.0" iyy="${shin_iyy}" iyz="0.0" izz="${shin_izz}"/>
+      </inertial>
+    </link>
+    <!-- Knee joint: thigh to shin -->
+    <joint name="${prefix}_knee" type="revolute">
+      <parent link="${prefix}_thigh_link"/>
+      <child link="${prefix}_shin_link"/>
+      <origin xyz="0 ${(thigh_radius + shin_radius + leg_offset) * reflect} ${-thigh_length/2}"/>
+      <axis xyz="0 1 0"/>
+      <limit lower="0" upper="2.36" effort="40" velocity="5"/>
     </joint>
   </xacro:macro>
@@ -149,8 +190,3 @@
   <xacro:leg prefix="right" reflect="-1" />
   <xacro:leg prefix="left" reflect="1" />
-  <joint name="base_to_head" type="fixed">
-    <parent link="base_link"/>
-    <child link="head_link"/>
-	<origin xyz="0 0 ${body_length}"/>
-  </joint>
 </robot>
