Commit message: Fix PR plane offset and use variables

File: models/environments/PR.xacro (robot description, xacro)
@@ -1,4 +1,13 @@
 <?xml version="1.0"?>
-<robot name="high_friction_plane">
+<robot xmlns:xacro="http://www.ros.org/wiki/xacro" name="high_friction_plane">
+  <!-- Plane properties -->
+  <xacro:property name="plane_length" value="10.0" />
+  <xacro:property name="plane_width" value="1.5" />
+  <xacro:property name="plane_height" value="0.1" />
+  <xacro:property name="plane_mass" value="10000" />
+  <xacro:property name="plane_ixx" value="1000" />
+  <xacro:property name="plane_iyy" value="1000" />
+  <xacro:property name="plane_izz" value="1000" />
+  <!-- Plane -->
   <link name="plane_link">
     <contact>
@@ -9,11 +18,11 @@
     <inertial>
       <origin xyz="0 0 0"/>
-      <mass value="10000"/> <!-- Massa muito alta para ser imóvel -->
-      <inertia ixx="1000" ixy="0" ixz="0" iyy="1000" iyz="0" izz="1000"/>
+      <mass value="${plane_mass}"/>
+      <inertia ixx="${plane_ixx}" ixy="0" ixz="0" iyy="${plane_iyy}" iyz="0" izz="${plane_izz}"/>
     </inertial>
     <visual>
-      <origin xyz="0 0 0"/>
+  <origin xyz="0 0 -${plane_height/2}"/>
       <geometry>
-        <box size="10.0 1.5 0.1"/> <!-- Comprimento (X) 10m, Largura (Y) 1.5m, Altura (Z) 0.1m -->
+        <box size="${plane_length} ${plane_width} ${plane_height}"/>
       </geometry>
       <material name="grey">
@@ -22,7 +31,7 @@
     </visual>
     <collision>
-      <origin xyz="0 0 0"/>
+  <origin xyz="0 0 -${plane_height/2}"/>
       <geometry>
-        <box size="10.0 1.5 0.1"/>
+        <box size="${plane_length} ${plane_width} ${plane_height}"/>
       </geometry>
     </collision>

Commit message: durante a ligacao2

File: models/environments/PR.xacro (robot description, xacro)
@@ -22,5 +22,5 @@
     </inertial>
     <visual>
-  <origin xyz="0 0 -${plane_height/2}"/>
+  <origin xyz="0 0 -${plane_height/2 - 0.3}"/>
       <geometry>
         <box size="${plane_length} ${plane_width} ${plane_height}"/>
@@ -31,5 +31,5 @@
     </visual>
     <collision>
-  <origin xyz="0 0 -${plane_height/2}"/>
+  <origin xyz="0 0 -${plane_height/2 - 0.3}"/>
       <geometry>
         <box size="${plane_length} ${plane_width} ${plane_height}"/>

File: models/robots/robot_stage1.xacro (robot description, xacro)
@@ -50,26 +50,29 @@
   </material>
   <!-- Body (main cylinder) -->
-  <link name="base_link">
+<link name="base_link">
+  <!-- CENTRO DE MASSA NO MEIO DO CORPO (Z = 0.45m) -->
+  <origin xyz="0 0 0"/>
+  <visual>
+    <!-- Alinha a geometria visual com o CM -->
+    <!-- Como o cilindro tem 0.6m de altura, e CM está no meio,
+         a base do cilindro fica em Z = 0.3 - 0.3 = 0.0 (no chão) -->
     <origin xyz="0 0 0"/>
-    <visual>
-      <!-- body_length/2 shifts the Z plane from the cylinder's center to its base -->
-      <!-- thigh_length + shin_length gives space for the legs -->
-      <origin xyz="0 0 ${body_length/2 + thigh_length + shin_length}"/>
-      <geometry>
-        <cylinder length="${body_length}" radius="${body_radius}"/>
-      </geometry>
-      <material name="robot_material"/>
-    </visual>
-    <collision>
-      <origin xyz="0 0 ${body_length/2 + thigh_length + shin_length}"/>
-      <geometry>
-        <cylinder length="${body_length}" radius="${body_radius}"/>
-      </geometry>
-    </collision>
-    <inertial>
-      <mass value="${body_mass}"/>
-      <inertia ixx="${body_ixx}" ixy="0.0" ixz="0.0" iyy="${body_iyy}" iyz="0.0" izz="${body_izz}"/>
-    </inertial>
-  </link>
+    <geometry>
+      <cylinder length="0.6" radius="0.2"/>
+    </geometry>
+    <material name="robot_material"/>
+  </visual>
+  <collision>
+    <!-- Mesma lógica: colisão alinhada ao CM -->
+    <origin xyz="0 0 0"/>
+    <geometry>
+      <cylinder length="0.6" radius="0.2"/>
+    </geometry>
+  </collision>
+  <inertial>
+    <mass value="2"/>
+    <inertia ixx="0.4" ixy="0.0" ixz="0.0" iyy="0.4" iyz="0.0" izz="0.2"/>
+  </inertial>
+</link>
   <!-- IMU (simulated sensor, offset from body center) -->
   <link name="imu_link">
@@ -99,5 +102,5 @@
     <!-- Z: Move the IMU body_length/3 to place it around the middle of the body -->
     <!-- X: Move the IMU body_radius to place it at the edge of the body -->
-    <origin xyz="${body_radius} 0 ${shin_length + thigh_length + body_length/3 }" rpy="0 0 0"/>
+    <origin xyz="0 0 0"/>
   </joint>
   <!-- Head (sphere) -->
