Commit message: Corrigir plano PR

File: environments/PR.xacro (robot description, xacro)
@@ -22,5 +22,5 @@
     </inertial>
     <visual>
-  <origin xyz="0 0 -${plane_height/2 - 0.3}"/>
+  <origin xyz="0 0 -${plane_height/2}"/>
       <geometry>
         <box size="${plane_length} ${plane_width} ${plane_height}"/>
@@ -31,5 +31,5 @@
     </visual>
     <collision>
-  <origin xyz="0 0 -${plane_height/2 - 0.3}"/>
+  <origin xyz="0 0 -${plane_height/2}"/>
       <geometry>
         <box size="${plane_length} ${plane_width} ${plane_height}"/>
