Commit message: Aumentar largura da pista para 2.5m

File: environments/PBA.xacro (robot description, xacro)
@@ -5,5 +5,5 @@
   <xacro:property name="middle_section_length" value="8.0" />
   <xacro:property name="final_section_length" value="1.0" />
-  <xacro:property name="plane_width" value="1.5" />
+  <xacro:property name="plane_width" value="2.5" />
   <xacro:property name="plane_height" value="0.1" />
   <xacro:property name="section_mass" value="10000" />

File: environments/PG.xacro (robot description, xacro)
@@ -5,5 +5,5 @@
   <xacro:property name="middle_section_length" value="8.0" />
   <xacro:property name="final_section_length" value="1.0" />
-  <xacro:property name="plane_width" value="1.5" />
+  <xacro:property name="plane_width" value="2.5" />
   <xacro:property name="plane_height" value="0.1" />
   <xacro:property name="section_mass" value="10000" />

File: environments/PR.xacro (robot description, xacro)
@@ -5,5 +5,5 @@
   <xacro:property name="middle_section_length" value="8.0" />
   <xacro:property name="final_section_length" value="1.0" />
-  <xacro:property name="plane_width" value="1.5" />
+  <xacro:property name="plane_width" value="2.5" />
   <xacro:property name="plane_height" value="0.1" />
   <xacro:property name="section_mass" value="10000" />

File: environments/PRA.xacro (robot description, xacro)
@@ -5,5 +5,5 @@
   <xacro:property name="middle_section_length" value="7.9156005496" /> <!-- cos(ramp_angle) * hypotenuse = cos(8.33 deg) * 8.0 -->
   <xacro:property name="final_section_length" value="1.0" />
-  <xacro:property name="plane_width" value="1.5" />
+  <xacro:property name="plane_width" value="2.5" />
   <xacro:property name="plane_height" value="0.1" />
   <xacro:property name="ramp_height" value="1.15899436545" /> <!-- sin(ramp_angle) * hypotenuse = sin(8.33 deg) * 8.0 -->

File: environments/PRB.xacro (robot description, xacro)
@@ -5,5 +5,5 @@
   <xacro:property name="middle_section_length" value="8.0" />
   <xacro:property name="final_section_length" value="1.0" />
-  <xacro:property name="plane_width" value="1.5" />
+  <xacro:property name="plane_width" value="2.5" />
   <xacro:property name="plane_height" value="0.1" />
   <xacro:property name="section_mass" value="10000" />

File: environments/PRD.xacro (robot description, xacro)
@@ -5,5 +5,5 @@
   <xacro:property name="middle_section_length" value="7.9156005496" /> <!-- cos(ramp_angle) * hypotenuse = cos(8.33 deg) * 8.0 -->
   <xacro:property name="final_section_length" value="1.0" />
-  <xacro:property name="plane_width" value="1.5" />
+  <xacro:property name="plane_width" value="2.5" />
   <xacro:property name="plane_height" value="0.1" />
   <xacro:property name="ramp_height" value="1.15899436545" /> <!-- sin(ramp_angle) * hypotenuse = sin(8.33 deg) * 8.0 -->

Commit message: Remover tags não suportadas pelo PyBullet

File: environments/PBA.xacro (robot description, xacro)
@@ -11,10 +11,4 @@
   <xacro:property name="section_iyy" value="1000" />
   <xacro:property name="section_izz" value="1000" />
-  <xacro:property name="pr_lateral_friction" value="0.8" />
-  <xacro:property name="pr_rolling_friction" value="0.0" />
-  <xacro:property name="pr_spinning_friction" value="0.0" />
-  <xacro:property name="pba_lateral_friction" value="0.5" />
-  <xacro:property name="pba_rolling_friction" value="0.8" />
-  <xacro:property name="pba_spinning_friction" value="1.0" />
   <!-- Materials -->
   <material name="initial_section_material">
@@ -29,9 +23,4 @@
   <!-- Base Link - Initial Section -->
   <link name="initial_link">
-    <contact>
-      <lateral_friction value="${pr_lateral_friction}"/>
-      <rolling_friction value="${pr_rolling_friction}"/>
-      <spinning_friction value="${pr_spinning_friction}"/>
-    </contact>
     <inertial>
       <origin xyz="0 0 -${plane_height/2}"/>
@@ -55,9 +44,4 @@
   <!-- Middle Section -->
   <link name="middle_link">
-    <contact>
-      <lateral_friction value="${pba_lateral_friction}"/>
-      <rolling_friction value="${pba_rolling_friction}"/>
-      <spinning_friction value="${pba_spinning_friction}"/>
-    </contact>
     <inertial>
       <origin xyz="0 0 -${plane_height/2}"/>
@@ -81,9 +65,4 @@
   <!-- Final Section -->
   <link name="final_link">
-    <contact>
-      <lateral_friction value="${pr_lateral_friction}"/>
-      <rolling_friction value="${pr_rolling_friction}"/>
-      <spinning_friction value="${pr_spinning_friction}"/>
-    </contact>
     <inertial>
       <origin xyz="0 0 -${plane_height/2}"/>

File: environments/PG.xacro (robot description, xacro)
@@ -11,10 +11,4 @@
   <xacro:property name="section_iyy" value="1000" />
   <xacro:property name="section_izz" value="1000" />
-  <xacro:property name="pr_lateral_friction" value="0.8" />
-  <xacro:property name="pr_rolling_friction" value="0.0" />
-  <xacro:property name="pr_spinning_friction" value="0.0" />
-  <xacro:property name="pg_lateral_friction" value="0.6" />
-  <xacro:property name="pg_rolling_friction" value="0.05" />
-  <xacro:property name="pg_spinning_friction" value="0.05" />
   <!-- Materials -->
   <material name="initial_section_material">
@@ -29,9 +23,4 @@
   <!-- Base Link - Initial Section -->
   <link name="initial_link">
-    <contact>
-      <lateral_friction value="${pr_lateral_friction}"/>
-      <rolling_friction value="${pr_rolling_friction}"/>
-      <spinning_friction value="${pr_spinning_friction}"/>
-    </contact>
     <inertial>
       <origin xyz="0 0 -${plane_height/2}"/>
@@ -55,9 +44,4 @@
   <!-- Middle Section -->
   <link name="middle_link">
-    <contact>
-      <lateral_friction value="${pg_lateral_friction}"/>
-      <rolling_friction value="${pg_rolling_friction}"/>
-      <spinning_friction value="${pg_spinning_friction}"/>
-    </contact>
     <inertial>
       <origin xyz="0 0 -${plane_height/2}"/>
@@ -81,9 +65,4 @@
   <!-- Final Section -->
   <link name="final_link">
-    <contact>
-      <lateral_friction value="${pr_lateral_friction}"/>
-      <rolling_friction value="${pr_rolling_friction}"/>
-      <spinning_friction value="${pr_spinning_friction}"/>
-    </contact>
     <inertial>
       <origin xyz="0 0 -${plane_height/2}"/>

File: environments/PR.xacro (robot description, xacro)
@@ -11,7 +11,4 @@
   <xacro:property name="section_iyy" value="1000" />
   <xacro:property name="section_izz" value="1000" />
-  <xacro:property name="lateral_friction" value="0.8" />
-  <xacro:property name="rolling_friction" value="0.0" />
-  <xacro:property name="spinning_friction" value="0.0" />
   <!-- Materials -->
   <material name="initial_section_material">
@@ -26,9 +23,4 @@
   <!-- Base Link - Initial Section -->
   <link name="initial_link">
-    <contact>
-      <lateral_friction value="${lateral_friction}"/>
-      <rolling_friction value="${rolling_friction}"/>
-      <spinning_friction value="${spinning_friction}"/>
-    </contact>
     <inertial>
       <origin xyz="0 0 -${plane_height/2}"/>
@@ -52,9 +44,4 @@
   <!-- Middle Section -->
   <link name="middle_link">
-    <contact>
-      <lateral_friction value="${lateral_friction}"/>
-      <rolling_friction value="${rolling_friction}"/>
-      <spinning_friction value="${spinning_friction}"/>
-    </contact>
     <inertial>
       <origin xyz="0 0 -${plane_height/2}"/>
@@ -78,9 +65,4 @@
   <!-- Final Section -->
   <link name="final_link">
-    <contact>
-      <lateral_friction value="${lateral_friction}"/>
-      <rolling_friction value="${rolling_friction}"/>
-      <spinning_friction value="${spinning_friction}"/>
-    </contact>
     <inertial>
       <origin xyz="0 0 -${plane_height/2}"/>

File: environments/PRA.xacro (robot description, xacro)
@@ -12,7 +12,4 @@
   <xacro:property name="section_iyy" value="1000" />
   <xacro:property name="section_izz" value="1000" />
-  <xacro:property name="pr_lateral_friction" value="0.8" />
-  <xacro:property name="pr_rolling_friction" value="0.0" />
-  <xacro:property name="pr_spinning_friction" value="0.0" />
   <!-- Materials -->
   <material name="initial_section_material">
@@ -27,9 +24,4 @@
   <!-- Base Link - Initial Section -->
   <link name="initial_link">
-    <contact>
-      <lateral_friction value="${pr_lateral_friction}"/>
-      <rolling_friction value="${pr_rolling_friction}"/>
-      <spinning_friction value="${pr_spinning_friction}"/>
-    </contact>
     <inertial>
       <origin xyz="0 0 -${plane_height/2}"/>
@@ -53,9 +45,4 @@
   <!-- Middle Section -->
   <link name="middle_link">
-    <contact>
-      <lateral_friction value="${pr_lateral_friction}"/>
-      <rolling_friction value="${pr_rolling_friction}"/>
-      <spinning_friction value="${pr_spinning_friction}"/>
-    </contact>
     <inertial>
       <origin xyz="0 0 0"/>
@@ -79,9 +66,4 @@
   <!-- Final Section -->
   <link name="final_link">
-    <contact>
-      <lateral_friction value="${pr_lateral_friction}"/>
-      <rolling_friction value="${pr_rolling_friction}"/>
-      <spinning_friction value="${pr_spinning_friction}"/>
-    </contact>
     <inertial>
       <origin xyz="0 0 -${plane_height/2}"/>

File: environments/PRB.xacro (robot description, xacro)
@@ -11,10 +11,4 @@
   <xacro:property name="section_iyy" value="1000" />
   <xacro:property name="section_izz" value="1000" />
-  <xacro:property name="pr_lateral_friction" value="0.8" />
-  <xacro:property name="pr_rolling_friction" value="0.0" />
-  <xacro:property name="pr_spinning_friction" value="0.0" />
-  <xacro:property name="prb_lateral_friction" value="0.8" />
-  <xacro:property name="prb_rolling_friction" value="0.0" />
-  <xacro:property name="prb_spinning_friction" value="0.0" />
   <!-- Materials -->
   <material name="initial_section_material">
@@ -29,9 +23,4 @@
   <!-- Base Link - Initial Section -->
   <link name="initial_link">
-    <contact>
-      <lateral_friction value="${pr_lateral_friction}"/>
-      <rolling_friction value="${pr_rolling_friction}"/>
-      <spinning_friction value="${pr_spinning_friction}"/>
-    </contact>
     <inertial>
       <origin xyz="0 0 -${plane_height/2}"/>
@@ -55,9 +44,4 @@
   <!-- Middle Section -->
   <link name="middle_link">
-    <contact>
-      <lateral_friction value="${prb_lateral_friction}"/>
-      <rolling_friction value="${prb_rolling_friction}"/>
-      <spinning_friction value="${prb_spinning_friction}"/>
-    </contact>
     <inertial>
       <origin xyz="0 0 -${plane_height/2}"/>
@@ -81,9 +65,4 @@
   <!-- Final Section -->
   <link name="final_link">
-    <contact>
-      <lateral_friction value="${pr_lateral_friction}"/>
-      <rolling_friction value="${pr_rolling_friction}"/>
-      <spinning_friction value="${pr_spinning_friction}"/>
-    </contact>
     <inertial>
       <origin xyz="0 0 -${plane_height/2}"/>

File: environments/PRD.xacro (robot description, xacro)
@@ -12,7 +12,4 @@
   <xacro:property name="section_iyy" value="1000" />
   <xacro:property name="section_izz" value="1000" />
-  <xacro:property name="pr_lateral_friction" value="0.8" />
-  <xacro:property name="pr_rolling_friction" value="0.0" />
-  <xacro:property name="pr_spinning_friction" value="0.0" />
   <!-- Materials -->
   <material name="initial_section_material">
@@ -27,9 +24,4 @@
   <!-- Base Link - Initial Section -->
   <link name="initial_link">
-    <contact>
-      <lateral_friction value="${pr_lateral_friction}"/>
-      <rolling_friction value="${pr_rolling_friction}"/>
-      <spinning_friction value="${pr_spinning_friction}"/>
-    </contact>
     <inertial>
       <origin xyz="0 0 -${plane_height/2}"/>
@@ -53,9 +45,4 @@
   <!-- Middle Section -->
   <link name="middle_link">
-    <contact>
-      <lateral_friction value="${pr_lateral_friction}"/>
-      <rolling_friction value="${pr_rolling_friction}"/>
-      <spinning_friction value="${pr_spinning_friction}"/>
-    </contact>
     <inertial>
       <origin xyz="0 0 0"/>
@@ -79,9 +66,4 @@
   <!-- Final Section -->
   <link name="final_link">
-    <contact>
-      <lateral_friction value="${pr_lateral_friction}"/>
-      <rolling_friction value="${pr_rolling_friction}"/>
-      <spinning_friction value="${pr_spinning_friction}"/>
-    </contact>
     <inertial>
       <origin xyz="0 0 -${plane_height/2}"/>
