Commit message: Arrumar parâmetros das rampas

File: environments/PRA.xacro (robot description, xacro)
@@ -3,9 +3,9 @@
   <!-- Plane properties -->
   <xacro:property name="initial_section_length" value="1.0" />
-  <xacro:property name="middle_section_length" value="8.0" />
+  <xacro:property name="middle_section_length" value="7.9156005496" /> <!-- cos(ramp_angle) * hypotenuse = cos(8.33 deg) * 8.0 -->
   <xacro:property name="final_section_length" value="1.0" />
   <xacro:property name="plane_width" value="1.5" />
   <xacro:property name="plane_height" value="0.1" />
-  <xacro:property name="ramp_height" value="2.14359353945" /> <!-- tan(ramp_angle) * ramp_length = tan(15 deg) * 8.0 -->
+  <xacro:property name="ramp_height" value="1.15899436545" /> <!-- sin(ramp_angle) * hypotenuse = sin(8.33 deg) * 8.0 -->
   <xacro:property name="section_mass" value="10000" />
   <xacro:property name="section_ixx" value="1000" />

File: environments/PRD.xacro (robot description, xacro)
@@ -3,9 +3,9 @@
   <!-- Plane properties -->
   <xacro:property name="initial_section_length" value="1.0" />
-  <xacro:property name="middle_section_length" value="8.0" />
+  <xacro:property name="middle_section_length" value="7.9156005496" /> <!-- cos(ramp_angle) * hypotenuse = cos(8.33 deg) * 8.0 -->
   <xacro:property name="final_section_length" value="1.0" />
   <xacro:property name="plane_width" value="1.5" />
   <xacro:property name="plane_height" value="0.1" />
-  <xacro:property name="ramp_height" value="2.14359353945" /> <!-- tan(ramp_angle) * ramp_length = tan(15 deg) * 8.0 -->
+  <xacro:property name="ramp_height" value="1.15899436545" /> <!-- sin(ramp_angle) * hypotenuse = sin(8.33 deg) * 8.0 -->
   <xacro:property name="section_mass" value="10000" />
   <xacro:property name="section_ixx" value="1000" />

Commit message: Corrigir rampas

File: environments/PRA.xacro (robot description, xacro)
@@ -8,4 +8,6 @@
   <xacro:property name="plane_height" value="0.1" />
   <xacro:property name="ramp_height" value="1.15899436545" /> <!-- sin(ramp_angle) * hypotenuse = sin(8.33 deg) * 8.0 -->
+  <xacro:property name="ramp_hypotenuse" value="8.0" />
+  <xacro:property name="ramp_angle_deg" value="8.33" />
   <xacro:property name="section_mass" value="10000" />
   <xacro:property name="section_ixx" value="1000" />

File: environments/PRD.xacro (robot description, xacro)
@@ -8,4 +8,6 @@
   <xacro:property name="plane_height" value="0.1" />
   <xacro:property name="ramp_height" value="1.15899436545" /> <!-- sin(ramp_angle) * hypotenuse = sin(8.33 deg) * 8.0 -->
+  <xacro:property name="ramp_hypotenuse" value="8.0" />
+  <xacro:property name="ramp_angle_deg" value="8.33" />
   <xacro:property name="section_mass" value="10000" />
   <xacro:property name="section_ixx" value="1000" />

Commit message: ajuste nas rampas

File: environments/PRA.xacro (robot description, xacro)
@@ -2,11 +2,11 @@
 <robot xmlns:xacro="http://www.ros.org/wiki/xacro" name="piso_rampa_ascendente">
   <!-- Plane properties -->
-  <xacro:property name="initial_section_length" value="1.0" />
-  <xacro:property name="middle_section_length" value="7.9156005496" /> <!-- cos(ramp_angle) * hypotenuse = cos(8.33 deg) * 8.0 -->
-  <xacro:property name="final_section_length" value="1.0" />
+  <xacro:property name="initial_section_length" value="1.037" />
+  <xacro:property name="middle_section_length" value="6.926" /> <!-- cos(ramp_angle) * hypotenuse = cos(8.33 deg) * 8.0 -->
+  <xacro:property name="final_section_length" value="1.037" />
   <xacro:property name="plane_width" value="2.5" />
   <xacro:property name="plane_height" value="0.1" />
-  <xacro:property name="ramp_height" value="1.15899436545" /> <!-- sin(ramp_angle) * hypotenuse = sin(8.33 deg) * 8.0 -->
-  <xacro:property name="ramp_hypotenuse" value="8.0" />
+  <xacro:property name="ramp_height" value="1.014" /> <!-- sin(ramp_angle) * hypotenuse = sin(8.33 deg) * 8.0 -->
+  <xacro:property name="ramp_hypotenuse" value="7.0" />
   <xacro:property name="ramp_angle_deg" value="8.33" />
   <xacro:property name="section_mass" value="10000" />

File: environments/PRD.xacro (robot description, xacro)
@@ -2,11 +2,11 @@
 <robot xmlns:xacro="http://www.ros.org/wiki/xacro" name="piso_rampa_descendente">
   <!-- Plane properties -->
-  <xacro:property name="initial_section_length" value="1.0" />
-  <xacro:property name="middle_section_length" value="7.9156005496" /> <!-- cos(ramp_angle) * hypotenuse = cos(8.33 deg) * 8.0 -->
-  <xacro:property name="final_section_length" value="1.0" />
+  <xacro:property name="initial_section_length" value="1.037" />
+  <xacro:property name="middle_section_length" value="6.926" /> <!-- cos(ramp_angle) * hypotenuse = cos(8.33 deg) * 8.0 -->
+  <xacro:property name="final_section_length" value="1.037" />
   <xacro:property name="plane_width" value="2.5" />
   <xacro:property name="plane_height" value="0.1" />
-  <xacro:property name="ramp_height" value="1.15899436545" /> <!-- sin(ramp_angle) * hypotenuse = sin(8.33 deg) * 8.0 -->
-  <xacro:property name="ramp_hypotenuse" value="8.0" />
+  <xacro:property name="ramp_height" value="1.014" /> <!-- sin(ramp_angle) * hypotenuse = sin(8.33 deg) * 8.0 -->
+  <xacro:property name="ramp_hypotenuse" value="7.0" />
   <xacro:property name="ramp_angle_deg" value="8.33" />
   <xacro:property name="section_mass" value="10000" />

Commit message: Revert "ajuste nas rampas"
This reverts commit 530654bc6786cb7b1a78b0552d4af17e81f68aec.

File: environments/PRA.xacro (robot description, xacro)
@@ -2,11 +2,11 @@
 <robot xmlns:xacro="http://www.ros.org/wiki/xacro" name="piso_rampa_ascendente">
   <!-- Plane properties -->
-  <xacro:property name="initial_section_length" value="1.037" />
-  <xacro:property name="middle_section_length" value="6.926" /> <!-- cos(ramp_angle) * hypotenuse = cos(8.33 deg) * 8.0 -->
-  <xacro:property name="final_section_length" value="1.037" />
+  <xacro:property name="initial_section_length" value="1.0" />
+  <xacro:property name="middle_section_length" value="7.9156005496" /> <!-- cos(ramp_angle) * hypotenuse = cos(8.33 deg) * 8.0 -->
+  <xacro:property name="final_section_length" value="1.0" />
   <xacro:property name="plane_width" value="2.5" />
   <xacro:property name="plane_height" value="0.1" />
-  <xacro:property name="ramp_height" value="1.014" /> <!-- sin(ramp_angle) * hypotenuse = sin(8.33 deg) * 8.0 -->
-  <xacro:property name="ramp_hypotenuse" value="7.0" />
+  <xacro:property name="ramp_height" value="1.15899436545" /> <!-- sin(ramp_angle) * hypotenuse = sin(8.33 deg) * 8.0 -->
+  <xacro:property name="ramp_hypotenuse" value="8.0" />
   <xacro:property name="ramp_angle_deg" value="8.33" />
   <xacro:property name="section_mass" value="10000" />

File: environments/PRD.xacro (robot description, xacro)
@@ -2,11 +2,11 @@
 <robot xmlns:xacro="http://www.ros.org/wiki/xacro" name="piso_rampa_descendente">
   <!-- Plane properties -->
-  <xacro:property name="initial_section_length" value="1.037" />
-  <xacro:property name="middle_section_length" value="6.926" /> <!-- cos(ramp_angle) * hypotenuse = cos(8.33 deg) * 8.0 -->
-  <xacro:property name="final_section_length" value="1.037" />
+  <xacro:property name="initial_section_length" value="1.0" />
+  <xacro:property name="middle_section_length" value="7.9156005496" /> <!-- cos(ramp_angle) * hypotenuse = cos(8.33 deg) * 8.0 -->
+  <xacro:property name="final_section_length" value="1.0" />
   <xacro:property name="plane_width" value="2.5" />
   <xacro:property name="plane_height" value="0.1" />
-  <xacro:property name="ramp_height" value="1.014" /> <!-- sin(ramp_angle) * hypotenuse = sin(8.33 deg) * 8.0 -->
-  <xacro:property name="ramp_hypotenuse" value="7.0" />
+  <xacro:property name="ramp_height" value="1.15899436545" /> <!-- sin(ramp_angle) * hypotenuse = sin(8.33 deg) * 8.0 -->
+  <xacro:property name="ramp_hypotenuse" value="8.0" />
   <xacro:property name="ramp_angle_deg" value="8.33" />
   <xacro:property name="section_mass" value="10000" />

Commit message: rampa a 4.16

File: environments/PRA.xacro (robot description, xacro)
@@ -3,11 +3,11 @@
   <!-- Plane properties -->
   <xacro:property name="initial_section_length" value="1.0" />
-  <xacro:property name="middle_section_length" value="7.9156005496" /> <!-- cos(ramp_angle) * hypotenuse = cos(8.33 deg) * 8.0 -->
+  <xacro:property name="middle_section_length" value="7.977656" /> <!-- cos(4.16 deg) -->
   <xacro:property name="final_section_length" value="1.0" />
   <xacro:property name="plane_width" value="2.5" />
   <xacro:property name="plane_height" value="0.1" />
-  <xacro:property name="ramp_height" value="1.15899436545" /> <!-- sin(ramp_angle) * hypotenuse = sin(8.33 deg) * 8.0 -->
+  <xacro:property name="ramp_height" value="0.580397" /> <!-- sin(4.16 deg) -->
   <xacro:property name="ramp_hypotenuse" value="8.0" />
-  <xacro:property name="ramp_angle_deg" value="8.33" />
+  <xacro:property name="ramp_angle_deg" value="4.16" />
   <xacro:property name="section_mass" value="10000" />
   <xacro:property name="section_ixx" value="1000" />

File: environments/PRD.xacro (robot description, xacro)
@@ -7,7 +7,7 @@
   <xacro:property name="plane_width" value="2.5" />
   <xacro:property name="plane_height" value="0.1" />
-  <xacro:property name="ramp_height" value="1.15899436545" /> <!-- sin(ramp_angle) * hypotenuse = sin(8.33 deg) * 8.0 -->
+  <xacro:property name="ramp_height" value="0.580397" /> <!-- sin(ramp_angle) * hypotenuse = sin(8.33 deg) * 8.0 -->
   <xacro:property name="ramp_hypotenuse" value="8.0" />
-  <xacro:property name="ramp_angle_deg" value="8.33" />
+  <xacro:property name="ramp_angle_deg" value="4.16" />
   <xacro:property name="section_mass" value="10000" />
   <xacro:property name="section_ixx" value="1000" />

Commit message: ajuste para 4.76

File: environments/PRA.xacro (robot description, xacro)
@@ -3,11 +3,11 @@
   <!-- Plane properties -->
   <xacro:property name="initial_section_length" value="1.0" />
-  <xacro:property name="middle_section_length" value="7.977656" /> <!-- cos(4.16 deg) -->
+  <xacro:property name="middle_section_length" value="7.972" /> <!-- cos(4.76 deg) -->
   <xacro:property name="final_section_length" value="1.0" />
   <xacro:property name="plane_width" value="2.5" />
   <xacro:property name="plane_height" value="0.1" />
-  <xacro:property name="ramp_height" value="0.580397" /> <!-- sin(4.16 deg) -->
+  <xacro:property name="ramp_height" value="0.664" /> <!-- sin(4.76 deg) -->
   <xacro:property name="ramp_hypotenuse" value="8.0" />
-  <xacro:property name="ramp_angle_deg" value="4.16" />
+  <xacro:property name="ramp_angle_deg" value="4.76" />
   <xacro:property name="section_mass" value="10000" />
   <xacro:property name="section_ixx" value="1000" />

File: environments/PRD.xacro (robot description, xacro)
@@ -3,11 +3,11 @@
   <!-- Plane properties -->
   <xacro:property name="initial_section_length" value="1.0" />
-  <xacro:property name="middle_section_length" value="7.9156005496" /> <!-- cos(ramp_angle) * hypotenuse = cos(8.33 deg) * 8.0 -->
+  <xacro:property name="middle_section_length" value="7.972" /> <!-- cos(ramp_angle) * hypotenuse = cos(8.33 deg) * 8.0 -->
   <xacro:property name="final_section_length" value="1.0" />
   <xacro:property name="plane_width" value="2.5" />
   <xacro:property name="plane_height" value="0.1" />
-  <xacro:property name="ramp_height" value="0.580397" /> <!-- sin(ramp_angle) * hypotenuse = sin(8.33 deg) * 8.0 -->
+  <xacro:property name="ramp_height" value="0.664" /> <!-- sin(ramp_angle) * hypotenuse = sin(8.33 deg) * 8.0 -->
   <xacro:property name="ramp_hypotenuse" value="8.0" />
-  <xacro:property name="ramp_angle_deg" value="4.16" />
+  <xacro:property name="ramp_angle_deg" value="4.76" />
   <xacro:property name="section_mass" value="10000" />
   <xacro:property name="section_ixx" value="1000" />
