Commit message: Aumentar amplitude do tornozelo

File: robots/robot_stage2.xacro (robot description, xacro)
@@ -246,5 +246,5 @@
       <origin xyz="0 0 ${-knee_radius - shin_length - ankle_radius}"/>
       <axis xyz="0 1 0"/>
-      <limit lower="${0 * deg_to_rad}" upper="${135 * deg_to_rad}" effort="40" velocity="5"/>
+      <limit lower="${-30 * deg_to_rad}" upper="${135 * deg_to_rad}" effort="40" velocity="5"/>
     </joint>
   </xacro:macro>

Commit message: salvei o robo 3 como 2 e coloquei braços no 3

File: robots/robot_stage2.xacro (robot description, xacro)
@@ -1,4 +1,4 @@
 <?xml version="1.0"?>
-<robot xmlns:xacro="http://www.ros.org/wiki/xacro" name="myrobot_st2">
+<robot xmlns:xacro="http://www.ros.org/wiki/xacro" name="myrobot_st3">
   <!-- Body properties -->
   <xacro:property name="body_radius" value="0.15" />
@@ -10,7 +10,11 @@
   <!-- Hip properties -->
   <xacro:property name="hip_radius" value="0.05" />
+  <xacro:property name="hip_mass" value="0.5" />
+  <xacro:property name="hip_ixx" value="0.01" />
+  <xacro:property name="hip_iyy" value="0.01" />
+  <xacro:property name="hip_izz" value="0.01" />
   <!-- Thigh properties -->
   <xacro:property name="thigh_radius" value="0.04" />
-  <xacro:property name="thigh_length" value="0.4" />
+  <xacro:property name="thigh_length" value="0.35" />
   <xacro:property name="thigh_mass" value="1.5" />
   <xacro:property name="thigh_ixx" value="0.02" />
@@ -19,8 +23,12 @@
   <!-- Knee properties -->
   <xacro:property name="knee_radius" value="0.04" />
+  <xacro:property name="knee_mass" value="0.5" />
+  <xacro:property name="knee_ixx" value="0.01" />
+  <xacro:property name="knee_iyy" value="0.01" />
+  <xacro:property name="knee_izz" value="0.01" />
   <!-- Shin properties -->
   <xacro:property name="shin_radius" value="0.035" />
   <xacro:property name="shin_length" value="0.30" />
-  <xacro:property name="shin_mass" value="1.0" />
+  <xacro:property name="shin_mass" value="1.5" />
   <xacro:property name="shin_ixx" value="0.015" />
   <xacro:property name="shin_iyy" value="0.015" />
@@ -28,10 +36,14 @@
   <!-- Ankle properties -->
   <xacro:property name="ankle_radius" value="0.03" />
+  <xacro:property name="ankle_mass" value="0.5" />
+  <xacro:property name="ankle_ixx" value="0.01" />
+  <xacro:property name="ankle_iyy" value="0.01" />
+  <xacro:property name="ankle_izz" value="0.01" />
   <!-- Foot properties -->
-  <xacro:property name="foot_length" value="0.2" />
-  <xacro:property name="foot_width" value="0.1" />
+  <xacro:property name="foot_length" value="0.35" />
+  <xacro:property name="foot_width" value="0.15" />
   <xacro:property name="foot_height" value="0.03" />
-  <xacro:property name="foot_offset_front" value="0.05" />
-  <xacro:property name="foot_mass" value="0.3" />
+  <xacro:property name="foot_offset_front" value="0.1" />
+  <xacro:property name="foot_mass" value="0.5" />
   <xacro:property name="foot_ixx" value="0.001" />
   <xacro:property name="foot_iyy" value="0.001" />
@@ -39,5 +51,5 @@
   <!-- Head properties -->
   <xacro:property name="head_radius" value="0.1" />
-  <xacro:property name="head_mass" value="0.2" />
+  <xacro:property name="head_mass" value="1.0" />
   <xacro:property name="head_ixx" value="0.005" />
   <xacro:property name="head_iyy" value="0.005" />
@@ -51,4 +63,7 @@
   <xacro:property name="imu_iyy" value="0.00001" />
   <xacro:property name="imu_izz" value="0.00001" />
+  <!-- Controle -->
+  <xacro:property name="joint_dumping" value="0.2" />
+  <xacro:property name="joint_friction" value="0.01" />
   <!-- Materials -->
   <material name="robot_material_1">
@@ -59,5 +74,5 @@
   </material>
   <!-- altura total -->
-  <xacro:property name="leg_total_length" value="${thigh_length + shin_length + 2 * ankle_radius + foot_height}" />
+  <xacro:property name="leg_total_length" value="${hip_radius + thigh_length + 2 * knee_radius + shin_length + 2 * ankle_radius + foot_height}" />
   <!-- body_offset: body_length/2 desloca o posicao Z do centro do cilindro (corpo do robo) para a sua base inferior, assim nao fica metade do corpo enterrado no chao -->
   <!-- body_offset: leg_total_length da espaco para as pernas, para elas nao ficarem enterradas no chao -->
@@ -82,4 +97,5 @@
     </collision>
     <inertial>
+      <origin xyz="0 0 ${body_offset}"/>
       <mass value="${body_mass}"/>
       <inertia ixx="${body_ixx}" ixy="0.0" ixz="0.0" iyy="${body_iyy}" iyz="0.0" izz="${body_izz}"/>
@@ -130,4 +146,5 @@
     </collision>
     <inertial>
+      <origin rpy="0 0 0" xyz="0 0 ${head_radius}"/>
       <mass value="${head_mass}"/>
       <inertia ixx="${head_ixx}" ixy="0.0" ixz="0.0" iyy="${head_iyy}" iyz="0.0" izz="${head_izz}"/>
@@ -144,4 +161,46 @@
   <!-- Leg macro (creates left/right leg: thigh, shin, foot) -->
   <xacro:macro name="leg" params="prefix reflect">
+    <!-- Hip joint: base_link to hip ball -->
+    <joint name="base_to_${prefix}_hip_ball" type="revolute">
+      <parent link="base_link"/>
+      <child link="${prefix}_hip_ball_link"/>
+      <!-- Z: Como o corpo principal e posicionado em 0 0 0, body_offset move o centro da esfera/articulacao para o centro do corpo -->
+      <!-- Z: Diminuir body_length/2 move o centro da esfera/articulacao para a base inferior do corpo -->
+      <!-- Y: body_radius posiciona o centro da esfera/articulacao do quadril na borda do corpo -->
+      <!-- Y: hip_radius tira a esfera/articulacao de dentro do corpo, caso contrario metade da esfera/articulacao ficaria dentro do corpo -->
+      <origin xyz="0 ${(body_radius + hip_radius) * reflect} ${body_offset - body_length/2}"/>
+      <axis xyz="0 1 0"/> <!-- Movimento frontal -->
+      <limit lower="${-90 * deg_to_rad}" upper="${90 * deg_to_rad}" effort="1000" velocity="5"/>
+      <dynamics damping="${joint_dumping}" friction="${joint_friction}"/>
+    </joint>
+    <!-- Hip Ball -->
+    <link name="${prefix}_hip_ball_link">
+      <visual>
+        <origin rpy="0 0 0" xyz="0 0 0"/>
+        <geometry>
+          <sphere radius="${hip_radius}"/>
+        </geometry>
+        <material name="robot_material_2"/>
+      </visual>
+      <collision>
+        <origin rpy="0 0 0" xyz="0 0 0"/>
+        <geometry>
+          <sphere radius="${hip_radius}"/>
+        </geometry>
+      </collision>
+      <inertial>
+        <mass value="${hip_mass}"/>
+        <inertia ixx="${hip_ixx}" ixy="0.0" ixz="0.0" iyy="${hip_iyy}" iyz="0.0" izz="${hip_izz}"/>
+      </inertial>
+    </link>
+    <!-- Hip joint: hip_ball_link to thigh -->
+    <joint name="hip_ball_to_${prefix}_thigh" type="revolute">
+      <parent link="${prefix}_hip_ball_link"/>
+      <child link="${prefix}_thigh_link"/>
+      <origin xyz="0 0 0"/>
+      <axis xyz="1 0 0"/> <!-- Movimento lateral -->
+      <limit lower="${-30 * deg_to_rad}" upper="${30 * deg_to_rad}" effort="1000" velocity="5"/>
+      <dynamics damping="${joint_dumping}" friction="${joint_friction}"/>
+    </joint>
     <!-- Thigh -->
     <link name="${prefix}_thigh_link">
@@ -162,20 +221,46 @@
       </collision>
       <inertial>
+        <origin rpy="0 0 0" xyz="0 0 ${-thigh_length/2 - hip_radius}"/>
         <mass value="${thigh_mass}"/>
         <inertia ixx="${thigh_ixx}" ixy="0.0" ixz="0.0" iyy="${thigh_iyy}" iyz="0.0" izz="${thigh_izz}"/>
       </inertial>
     </link>
-    <!-- Hip joint: base_link to thigh -->
-    <joint name="base_to_${prefix}_thigh" type="revolute">
-      <parent link="base_link"/>
-      <child link="${prefix}_thigh_link"/>
-      <!-- Z: Como o corpo principal e posicionado em 0 0 0, body_offset move o centro da esfera/articulacao para o centro do corpo -->
-      <!-- Z: Diminuir body_length/2 move o centro da esfera/articulacao para a base inferior do corpo -->
-      <!-- Z: Somar hip_radius faz a base inferior da esfera/articulacao do quadril coincidir com a base inferior do corpo -->
-      <!-- Y: body_radius posiciona o centro da esfera/articulacao do quadril na borda do corpo -->
-      <!-- Y: hip_radius tira a esfera/articulacao de dentro do corpo, caso contrario metade da esfera/articulacao ficaria dentro do corpo -->
-      <origin xyz="0 ${(body_radius + hip_radius) * reflect} ${body_offset - body_length/2 + hip_radius}"/>
+    <!-- Knee joint: thigh to knee ball -->
+    <joint name="${prefix}_thigh_to_knee_ball" type="fixed">
+      <parent link="${prefix}_thigh_link"/>
+      <child link="${prefix}_knee_ball_link"/>
+      <!-- Z: Como o parent e a coxa, o centro da esfera/articulacao do joelho coincide inicialmente com sua referencia que é o hip joint posicionado na base inferior do body -->
+      <!-- Z: Diminuir hip_radius + thigh_length faz o centro da esfera/articulacao do joelho coincidir com a base inferior da coxa -->
+      <!-- Z: Diminuir knee_radius faz o topo da esfera/articulacao do joelho coincidir com a base inferior da coxa -->
+      <origin xyz="0 0 ${-hip_radius - thigh_length - knee_radius }"/>
+    </joint>
+    <!-- Knee Ball -->
+    <link name="${prefix}_knee_ball_link">
+      <visual>
+        <origin rpy="0 0 0" xyz="0 0 0"/>
+        <geometry>
+          <sphere radius="${knee_radius}"/>
+        </geometry>
+        <material name="robot_material_2"/>
+      </visual>
+      <collision>
+        <origin rpy="0 0 0" xyz="0 0 0"/>
+        <geometry>
+          <sphere radius="${knee_radius}"/>
+        </geometry>
+      </collision>
+      <inertial>
+        <mass value="${knee_mass}"/>
+        <inertia ixx="${knee_ixx}" ixy="0.0" ixz="0.0" iyy="${knee_iyy}" iyz="0.0" izz="${knee_izz}"/>
+      </inertial>
+    </link>
+    <!-- Knee joint: knee ball to shin -->
+    <joint name="${prefix}_knee_ball_to_shin" type="revolute">
+      <parent link="${prefix}_knee_ball_link"/>
+      <child link="${prefix}_shin_link"/>
+      <origin xyz="0 0 0"/>
       <axis xyz="0 1 0"/>
-      <limit lower="${-90 * deg_to_rad}" upper="${90 * deg_to_rad}" effort="50" velocity="5"/>
+      <limit lower="${0 * deg_to_rad}" upper="${135 * deg_to_rad}" effort="1000" velocity="5"/>
+      <dynamics damping="${joint_dumping}" friction="${joint_friction}"/>
     </joint>
     <!-- Shin -->
@@ -197,20 +282,46 @@
       </collision>
       <inertial>
+        <origin rpy="0 0 0" xyz="0 0 ${-shin_length/2 - knee_radius}"/>
         <mass value="${shin_mass}"/>
         <inertia ixx="${shin_ixx}" ixy="0.0" ixz="0.0" iyy="${shin_iyy}" iyz="0.0" izz="${shin_izz}"/>
       </inertial>
     </link>
-    <!-- Knee joint: thigh to shin -->
-    <joint name="${prefix}_knee" type="revolute">
-      <parent link="${prefix}_thigh_link"/>
-      <child link="${prefix}_shin_link"/>
-      <!-- Z: Como o parent e a coxa, o centro da esfera/articulacao do joelho coincide inicialmente com o centro da esfera/articulacao do quadril -->
-      <!-- Z: Diminuir hip_radius + thigh_length faz o centro da esfera/articulacao do joelho coincidir com a base inferior da coxa -->
-      <!-- Z: Somar knee_radius faz a base inferior da esfera/articulacao do joelho coincidir com a base inferior da coxa -->
-      <!-- Y: thigh_radius posiciona o centro esfera/articulacao do joelho na borda da coxa -->
-      <!-- Y: knee_radius tira a esfera/articulacao de dentro da coxa, caso contrario metade da esfera/articulacao ficaria dentro da coxa -->
-      <origin xyz="0 ${(-thigh_radius + -knee_radius) * reflect} ${-hip_radius - thigh_length + knee_radius}"/>
+    <!-- Ankle joint: shin to ankle ball -->
+    <joint name="${prefix}_shin_to_ankle_ball" type="fixed">
+      <parent link="${prefix}_shin_link"/>
+      <child link="${prefix}_ankle_ball_link"/>
+      <!-- Z: Como o parent e a canela, o centro da esfera/articulacao do tornozelo coincide inicialmente com sua referencia que é o knee joint -->
+      <!-- Z: Diminuir knee_radius + shin_length faz o centro da esfera/articulacao do tornozelo coincidir com a base inferior da canela -->
+      <!-- Z: Diminuir ankle_radius faz o topo da esfera/articulacao do tornozelo coincidir com a base inferior da canela -->
+      <origin xyz="0 0 ${-knee_radius - shin_length - ankle_radius}"/>
+    </joint>
+    <!-- Ankle Ball -->
+    <link name="${prefix}_ankle_ball_link">
+      <visual>
+        <origin rpy="0 0 0" xyz="0 0 0"/>
+        <geometry>
+          <sphere radius="${ankle_radius}"/>
+        </geometry>
+        <material name="robot_material_2"/>
+      </visual>
+      <collision>
+        <origin rpy="0 0 0" xyz="0 0 0"/>
+        <geometry>
+          <sphere radius="${ankle_radius}"/>
+        </geometry>
+      </collision>
+      <inertial>
+        <mass value="${ankle_mass}"/>
+        <inertia ixx="${ankle_ixx}" ixy="0.0" ixz="0.0" iyy="${ankle_iyy}" iyz="0.0" izz="${ankle_izz}"/>
+      </inertial>
+    </link>
+    <!-- Ankle joint: ankle ball to foot -->
+    <joint name="${prefix}_ankle_ball_to_foot" type="revolute">
+      <parent link="${prefix}_ankle_ball_link"/>
+      <child link="${prefix}_foot_link"/>
+      <origin xyz="0 0 0"/>
       <axis xyz="0 1 0"/>
-      <limit lower="${0 * deg_to_rad}" upper="${135 * deg_to_rad}" effort="40" velocity="5"/>
+      <limit lower="${-30 * deg_to_rad}" upper="${75 * deg_to_rad}" effort="1000" velocity="5"/>
+      <dynamics damping="${joint_dumping}" friction="${joint_friction}"/>
     </joint>
     <!-- Foot -->
@@ -233,19 +344,9 @@
       </collision>
       <inertial>
+        <origin rpy="0 0 0" xyz="${foot_offset_front} 0 ${-ankle_radius - foot_height/2}"/>
         <mass value="${foot_mass}"/>
         <inertia ixx="${foot_ixx}" ixy="0.0" ixz="0.0" iyy="${foot_iyy}" iyz="0.0" izz="${foot_izz}"/>
       </inertial>
     </link>
-    <!-- Ankle joint: shin to foot -->
-    <joint name="${prefix}_ankle_joint" type="revolute">
-      <parent link="${prefix}_shin_link"/>
-      <child link="${prefix}_foot_link"/>
-      <!-- Z: Como o parent e a canela, o centro da esfera/articulacao do tornozelo coincide inicialmente com o centro da esfera/articulacao do joelho -->
-      <!-- Z: Diminuir knee_radius + shin_length faz o centro da esfera/articulacao do tornozelo coincidir com a base inferior da canela -->
-      <!-- Z: Diminuir ankle_radius faz a base superior da esfera/articulacao do tornozelo coincidir com a base inferior da canela -->
-      <origin xyz="0 0 ${-knee_radius - shin_length - ankle_radius}"/>
-      <axis xyz="0 1 0"/>
-      <limit lower="${-30 * deg_to_rad}" upper="${135 * deg_to_rad}" effort="40" velocity="5"/>
-    </joint>
   </xacro:macro>
   <!-- Instantiate right and left legs -->

File: robots/robot_stage3.xacro (robot description, xacro)
@@ -353,3 +353,142 @@
   <xacro:leg prefix="right" reflect="-1" />
   <xacro:leg prefix="left" reflect="1" />
+  <!-- Shoulder properties -->
+<xacro:property name="shoulder_radius" value="0.04" />
+<xacro:property name="shoulder_length" value="0.1" />
+<xacro:property name="shoulder_mass" value="0.3" />
+<!-- Upper arm properties -->
+<xacro:property name="upper_arm_radius" value="0.035" />
+<xacro:property name="upper_arm_length" value="0.25" />
+<xacro:property name="upper_arm_mass" value="0.8" />
+<!-- Lower arm properties -->
+<xacro:property name="lower_arm_radius" value="0.03" />
+<xacro:property name="lower_arm_length" value="0.22" />
+<xacro:property name="lower_arm_mass" value="0.6" />
+<!-- Hand properties -->
+<xacro:property name="hand_length" value="0.08" />
+<xacro:property name="hand_width" value="0.06" />
+<xacro:property name="hand_height" value="0.04" />
+<xacro:property name="hand_mass" value="0.2" />
+<!-- Arm macro -->
+<xacro:macro name="arm" params="prefix reflect">
+  <!-- Shoulder joint: base_link to shoulder -->
+  <joint name="base_to_${prefix}_shoulder" type="revolute">
+    <parent link="base_link"/>
+    <child link="${prefix}_shoulder_link"/>
+    <origin xyz="0 ${(body_radius + shoulder_radius) * reflect} ${body_offset + body_length/4}" rpy="0 0 0"/>
+    <axis xyz="0 1 0"/> <!-- Shoulder abduction/adduction -->
+    <limit lower="${-90 * deg_to_rad}" upper="${90 * deg_to_rad}" effort="100" velocity="3"/>
+    <dynamics damping="0.1" friction="0.01"/>
+  </joint>
+  <!-- Shoulder link -->
+  <link name="${prefix}_shoulder_link">
+    <visual>
+      <origin rpy="0 0 0" xyz="0 0 0"/>
+      <geometry>
+        <sphere radius="${shoulder_radius}"/>
+      </geometry>
+      <material name="robot_material_2"/>
+    </visual>
+    <collision>
+      <origin rpy="0 0 0" xyz="0 0 0"/>
+      <geometry>
+        <sphere radius="${shoulder_radius}"/>
+      </geometry>
+    </collision>
+    <inertial>
+      <mass value="${shoulder_mass}"/>
+      <inertia ixx="0.001" ixy="0.0" ixz="0.0" iyy="0.001" iyz="0.0" izz="0.001"/>
+    </inertial>
+  </link>
+  <!-- Upper arm joint: shoulder to upper arm -->
+  <joint name="${prefix}_shoulder_to_upper_arm" type="revolute">
+    <parent link="${prefix}_shoulder_link"/>
+    <child link="${prefix}_upper_arm_link"/>
+    <origin xyz="0 0 0" rpy="0 0 0"/>
+    <axis xyz="1 0 0"/> <!-- Shoulder flexion/extension -->
+    <limit lower="${-120 * deg_to_rad}" upper="${30 * deg_to_rad}" effort="80" velocity="3"/>
+    <dynamics damping="0.1" friction="0.01"/>
+  </joint>
+  <!-- Upper arm link -->
+  <link name="${prefix}_upper_arm_link">
+    <visual>
+      <origin rpy="0 ${90 * deg_to_rad} 0" xyz="0 0 ${-upper_arm_length/2}"/>
+      <geometry>
+        <cylinder length="${upper_arm_length}" radius="${upper_arm_radius}"/>
+      </geometry>
+      <material name="robot_material_1"/>
+    </visual>
+    <collision>
+      <origin rpy="0 ${90 * deg_to_rad} 0" xyz="0 0 ${-upper_arm_length/2}"/>
+      <geometry>
+        <cylinder length="${upper_arm_length}" radius="${upper_arm_radius}"/>
+      </geometry>
+    </collision>
+    <inertial>
+      <origin rpy="0 ${90 * deg_to_rad} 0" xyz="0 0 ${-upper_arm_length/2}"/>
+      <mass value="${upper_arm_mass}"/>
+      <inertia ixx="0.005" ixy="0.0" ixz="0.0" iyy="0.005" iyz="0.0" izz="0.001"/>
+    </inertial>
+  </link>
+  <!-- Elbow joint: upper arm to lower arm -->
+  <joint name="${prefix}_upper_arm_to_lower_arm" type="revolute">
+    <parent link="${prefix}_upper_arm_link"/>
+    <child link="${prefix}_lower_arm_link"/>
+    <origin xyz="0 0 ${-upper_arm_length}" rpy="0 0 0"/>
+    <axis xyz="1 0 0"/> <!-- Elbow flexion/extension -->
+    <limit lower="${0 * deg_to_rad}" upper="${150 * deg_to_rad}" effort="60" velocity="3"/>
+    <dynamics damping="0.1" friction="0.01"/>
+  </joint>
+  <!-- Lower arm link -->
+  <link name="${prefix}_lower_arm_link">
+    <visual>
+      <origin rpy="0 ${90 * deg_to_rad} 0" xyz="0 0 ${-lower_arm_length/2}"/>
+      <geometry>
+        <cylinder length="${lower_arm_length}" radius="${lower_arm_radius}"/>
+      </geometry>
+      <material name="robot_material_1"/>
+    </visual>
+    <collision>
+      <origin rpy="0 ${90 * deg_to_rad} 0" xyz="0 0 ${-lower_arm_length/2}"/>
+      <geometry>
+        <cylinder length="${lower_arm_length}" radius="${lower_arm_radius}"/>
+      </geometry>
+    </collision>
+    <inertial>
+      <origin rpy="0 ${90 * deg_to_rad} 0" xyz="0 0 ${-lower_arm_length/2}"/>
+      <mass value="${lower_arm_mass}"/>
+      <inertia ixx="0.003" ixy="0.0" ixz="0.0" iyy="0.003" iyz="0.0" izz="0.001"/>
+    </inertial>
+  </link>
+  <!-- Hand joint: lower arm to hand -->
+  <joint name="${prefix}_lower_arm_to_hand" type="fixed">
+    <parent link="${prefix}_lower_arm_link"/>
+    <child link="${prefix}_hand_link"/>
+    <origin xyz="0 0 ${-lower_arm_length}" rpy="0 0 0"/>
+  </joint>
+  <!-- Hand link -->
+  <link name="${prefix}_hand_link">
+    <visual>
+      <origin rpy="0 0 0" xyz="0 0 ${-hand_height/2}"/>
+      <geometry>
+        <box size="${hand_length} ${hand_width} ${hand_height}"/>
+      </geometry>
+      <material name="robot_material_2"/>
+    </visual>
+    <collision>
+      <origin rpy="0 0 0" xyz="0 0 ${-hand_height/2}"/>
+      <geometry>
+        <box size="${hand_length} ${hand_width} ${hand_height}"/>
+      </geometry>
+    </collision>
+    <inertial>
+      <origin rpy="0 0 0" xyz="0 0 ${-hand_height/2}"/>
+      <mass value="${hand_mass}"/>
+      <inertia ixx="0.0001" ixy="0.0" ixz="0.0" iyy="0.0001" iyz="0.0" izz="0.0001"/>
+    </inertial>
+  </link>
+</xacro:macro>
+<!-- Instantiate arms -->
+<xacro:arm prefix="right" reflect="-1"/>
+<xacro:arm prefix="left" reflect="1"/>
 </robot>
