Commit message: Ajustar centro de massa e script pre fill

File: robots/robot_stage3.xacro (robot description, xacro)
@@ -30,5 +30,5 @@
   <xacro:property name="shin_radius" value="0.035" />
   <xacro:property name="shin_length" value="0.30" />
-  <xacro:property name="shin_mass" value="1.0" />
+  <xacro:property name="shin_mass" value="1.5" />
   <xacro:property name="shin_ixx" value="0.015" />
   <xacro:property name="shin_iyy" value="0.015" />
@@ -41,9 +41,9 @@
   <xacro:property name="ankle_izz" value="0.01" />
   <!-- Foot properties -->
-  <xacro:property name="foot_length" value="0.2" />
-  <xacro:property name="foot_width" value="0.1" />
+  <xacro:property name="foot_length" value="0.35" />
+  <xacro:property name="foot_width" value="0.15" />
   <xacro:property name="foot_height" value="0.03" />
-  <xacro:property name="foot_offset_front" value="0.05" />
-  <xacro:property name="foot_mass" value="0.3" />
+  <xacro:property name="foot_offset_front" value="0.1" />
+  <xacro:property name="foot_mass" value="0.5" />
   <xacro:property name="foot_ixx" value="0.001" />
   <xacro:property name="foot_iyy" value="0.001" />
@@ -51,5 +51,5 @@
   <!-- Head properties -->
   <xacro:property name="head_radius" value="0.1" />
-  <xacro:property name="head_mass" value="0.2" />
+  <xacro:property name="head_mass" value="1.0" />
   <xacro:property name="head_ixx" value="0.005" />
   <xacro:property name="head_iyy" value="0.005" />
@@ -97,4 +97,5 @@
     </collision>
     <inertial>
+      <origin xyz="0 0 ${body_offset}"/>
       <mass value="${body_mass}"/>
       <inertia ixx="${body_ixx}" ixy="0.0" ixz="0.0" iyy="${body_iyy}" iyz="0.0" izz="${body_izz}"/>
@@ -145,4 +146,5 @@
     </collision>
     <inertial>
+      <origin rpy="0 0 0" xyz="0 0 ${head_radius}"/>
       <mass value="${head_mass}"/>
       <inertia ixx="${head_ixx}" ixy="0.0" ixz="0.0" iyy="${head_iyy}" iyz="0.0" izz="${head_izz}"/>
@@ -219,4 +221,5 @@
       </collision>
       <inertial>
+        <origin rpy="0 0 0" xyz="0 0 ${-thigh_length/2 - hip_radius}"/>
         <mass value="${thigh_mass}"/>
         <inertia ixx="${thigh_ixx}" ixy="0.0" ixz="0.0" iyy="${thigh_iyy}" iyz="0.0" izz="${thigh_izz}"/>
@@ -279,4 +282,5 @@
       </collision>
       <inertial>
+        <origin rpy="0 0 0" xyz="0 0 ${-shin_length/2 - knee_radius}"/>
         <mass value="${shin_mass}"/>
         <inertia ixx="${shin_ixx}" ixy="0.0" ixz="0.0" iyy="${shin_iyy}" iyz="0.0" izz="${shin_izz}"/>
@@ -340,4 +344,5 @@
       </collision>
       <inertial>
+        <origin rpy="0 0 0" xyz="${foot_offset_front} 0 ${-ankle_radius - foot_height/2}"/>
         <mass value="${foot_mass}"/>
         <inertia ixx="${foot_ixx}" ixy="0.0" ixz="0.0" iyy="${foot_iyy}" iyz="0.0" izz="${foot_izz}"/>

Commit message: Renomear dumping para damping

File: robots/robot_stage3.xacro (robot description, xacro)
@@ -64,5 +64,5 @@
   <xacro:property name="imu_izz" value="0.00001" />
   <!-- Controle -->
-  <xacro:property name="joint_dumping" value="0.2" />
+  <xacro:property name="joint_damping" value="0.2" />
   <xacro:property name="joint_friction" value="0.01" />
   <!-- Materials -->
@@ -172,5 +172,5 @@
       <axis xyz="0 1 0"/> <!-- Movimento frontal -->
       <limit lower="${-90 * deg_to_rad}" upper="${90 * deg_to_rad}" effort="1000" velocity="5"/>
-      <dynamics damping="${joint_dumping}" friction="${joint_friction}"/>
+      <dynamics damping="${joint_damping}" friction="${joint_friction}"/>
     </joint>
     <!-- Hip Ball -->
@@ -201,5 +201,5 @@
       <axis xyz="1 0 0"/> <!-- Movimento lateral -->
       <limit lower="${-30 * deg_to_rad}" upper="${30 * deg_to_rad}" effort="1000" velocity="5"/>
-      <dynamics damping="${joint_dumping}" friction="${joint_friction}"/>
+      <dynamics damping="${joint_damping}" friction="${joint_friction}"/>
     </joint>
     <!-- Thigh -->
@@ -262,5 +262,5 @@
       <axis xyz="0 1 0"/>
       <limit lower="${0 * deg_to_rad}" upper="${135 * deg_to_rad}" effort="1000" velocity="5"/>
-      <dynamics damping="${joint_dumping}" friction="${joint_friction}"/>
+      <dynamics damping="${joint_damping}" friction="${joint_friction}"/>
     </joint>
     <!-- Shin -->
@@ -323,5 +323,5 @@
       <axis xyz="0 1 0"/>
       <limit lower="${-30 * deg_to_rad}" upper="${75 * deg_to_rad}" effort="1000" velocity="5"/>
-      <dynamics damping="${joint_dumping}" friction="${joint_friction}"/>
+      <dynamics damping="${joint_damping}" friction="${joint_friction}"/>
     </joint>
     <!-- Foot -->

File: robots/robot_stage4.xacro (robot description, xacro)
@@ -64,5 +64,5 @@
   <xacro:property name="imu_izz" value="0.00001" />
   <!-- Controle -->
-  <xacro:property name="joint_dumping" value="0.2" />
+  <xacro:property name="joint_damping" value="0.2" />
   <xacro:property name="joint_friction" value="0.01" />
   <!-- Materials -->
@@ -172,5 +172,5 @@
       <axis xyz="0 1 0"/> <!-- Movimento frontal -->
       <limit lower="${-75 * deg_to_rad}" upper="${60 * deg_to_rad}" effort="1000" velocity="5"/>
-      <dynamics damping="${joint_dumping}" friction="${joint_friction}"/>
+      <dynamics damping="${joint_damping}" friction="${joint_friction}"/>
     </joint>
     <!-- Hip Ball -->
@@ -201,5 +201,5 @@
       <axis xyz="1 0 0"/> <!-- Movimento lateral -->
       <limit lower="${-30 * deg_to_rad}" upper="${30 * deg_to_rad}" effort="1000" velocity="5"/>
-      <dynamics damping="${joint_dumping}" friction="${joint_friction}"/>
+      <dynamics damping="${joint_damping}" friction="${joint_friction}"/>
     </joint>
     <!-- Thigh -->
@@ -262,5 +262,5 @@
       <axis xyz="0 1 0"/>
       <limit lower="${0 * deg_to_rad}" upper="${90 * deg_to_rad}" effort="1000" velocity="5"/>
-      <dynamics damping="${joint_dumping}" friction="${joint_friction}"/>
+      <dynamics damping="${joint_damping}" friction="${joint_friction}"/>
     </joint>
     <!-- Shin -->
@@ -297,5 +297,5 @@
       <axis xyz="0 1 0"/> <!-- Movimento frontal -->
       <limit lower="${-30 * deg_to_rad}" upper="${75 * deg_to_rad}" effort="1000" velocity="5"/>
-      <dynamics damping="${joint_dumping}" friction="${joint_friction}"/>
+      <dynamics damping="${joint_damping}" friction="${joint_friction}"/>
     </joint>
     <!-- Ankle Ball -->
@@ -326,5 +326,5 @@
       <axis xyz="1 0 0"/> <!-- Movimento lateral -->
       <limit lower="${-30 * deg_to_rad}" upper="${30 * deg_to_rad}" effort="1000" velocity="5"/>
-      <dynamics damping="${joint_dumping}" friction="${joint_friction}"/>
+      <dynamics damping="${joint_damping}" friction="${joint_friction}"/>
     </joint>
     <!-- Foot -->

File: robots/robot_stage5.xacro (robot description, xacro)
@@ -93,5 +93,5 @@
   <xacro:property name="imu_izz" value="0.00001" />
   <!-- Controle -->
-  <xacro:property name="joint_dumping" value="0.2" />
+  <xacro:property name="joint_damping" value="0.2" />
   <xacro:property name="joint_friction" value="0.01" />
   <!-- Materials -->
@@ -201,5 +201,5 @@
       <axis xyz="0 1 0"/> <!-- Movimento frontal -->
       <limit lower="${-75 * deg_to_rad}" upper="${60 * deg_to_rad}" effort="1000" velocity="5"/>
-      <dynamics damping="${joint_dumping}" friction="${joint_friction}"/>
+      <dynamics damping="${joint_damping}" friction="${joint_friction}"/>
     </joint>
     <!-- Hip Ball -->
@@ -230,5 +230,5 @@
       <axis xyz="1 0 0"/> <!-- Movimento lateral -->
       <limit lower="${-30 * deg_to_rad}" upper="${30 * deg_to_rad}" effort="1000" velocity="5"/>
-      <dynamics damping="${joint_dumping}" friction="${joint_friction}"/>
+      <dynamics damping="${joint_damping}" friction="${joint_friction}"/>
     </joint>
     <!-- Thigh -->
@@ -291,5 +291,5 @@
       <axis xyz="0 1 0"/>
       <limit lower="${0 * deg_to_rad}" upper="${90 * deg_to_rad}" effort="1000" velocity="5"/>
-      <dynamics damping="${joint_dumping}" friction="${joint_friction}"/>
+      <dynamics damping="${joint_damping}" friction="${joint_friction}"/>
     </joint>
     <!-- Shin -->
@@ -326,5 +326,5 @@
       <axis xyz="0 1 0"/> <!-- Movimento frontal -->
       <limit lower="${-30 * deg_to_rad}" upper="${75 * deg_to_rad}" effort="1000" velocity="5"/>
-      <dynamics damping="${joint_dumping}" friction="${joint_friction}"/>
+      <dynamics damping="${joint_damping}" friction="${joint_friction}"/>
     </joint>
     <!-- Ankle Ball -->
@@ -355,5 +355,5 @@
       <axis xyz="1 0 0"/> <!-- Movimento lateral -->
       <limit lower="${-30 * deg_to_rad}" upper="${30 * deg_to_rad}" effort="1000" velocity="5"/>
-      <dynamics damping="${joint_dumping}" friction="${joint_friction}"/>
+      <dynamics damping="${joint_damping}" friction="${joint_friction}"/>
     </joint>
     <!-- Foot -->
@@ -395,5 +395,5 @@
     <!-- Limite de 45° para frente e trás -->
     <limit lower="${-45 * deg_to_rad}" upper="${45 * deg_to_rad}" effort="100" velocity="3"/>
-    <dynamics damping="${joint_dumping}" friction="${joint_friction}"/>
+    <dynamics damping="${joint_damping}" friction="${joint_friction}"/>
   </joint>
   <!-- Shoulder frontal link -->
@@ -425,5 +425,5 @@
     <!-- Limitar movimento lateral -->
     <limit lower="${-10 * deg_to_rad}" upper="${45 * deg_to_rad}" effort="80" velocity="3"/>
-    <dynamics damping="${joint_dumping}" friction="${joint_friction}"/>
+    <dynamics damping="${joint_damping}" friction="${joint_friction}"/>
   </joint>
   <!-- Shoulder lateral link -->
