Commit message: inclui alteração do robot, graficos aparecem.

File: robots/robot_stage1.xacro (robot description, xacro)
@@ -2,65 +2,65 @@
 <robot xmlns:xacro="http://www.ros.org/wiki/xacro" name="myrobot">
   <!-- Body properties -->
-  <xacro:property name="body_radius" value="0.2" />
-  <xacro:property name="body_length" value="0.6" />
-  <xacro:property name="body_mass" value="2" />
-  <xacro:property name="body_ixx" value="0.4" />
-  <xacro:property name="body_iyy" value="0.4" />
-  <xacro:property name="body_izz" value="0.2" />
+  <xacro:property name="body_radius" value="0.15" />
+  <xacro:property name="body_length" value="0.3" />
+  <xacro:property name="body_mass" value="5.0" />
+  <xacro:property name="body_ixx" value="0.1" />
+  <xacro:property name="body_iyy" value="0.1" />
+  <xacro:property name="body_izz" value="0.05" />
   <!-- Hip properties -->
-  <xacro:property name="hip_radius" value="0.1" />
+  <xacro:property name="hip_radius" value="0.05" />
   <!-- Thigh properties -->
-  <xacro:property name="thigh_radius" value="0.1" />
-  <xacro:property name="thigh_length" value="0.35" />
-  <xacro:property name="thigh_mass" value="2" />
+  <xacro:property name="thigh_radius" value="0.04" />
+  <xacro:property name="thigh_length" value="0.4" />
+  <xacro:property name="thigh_mass" value="1.5" />
   <xacro:property name="thigh_ixx" value="0.02" />
   <xacro:property name="thigh_iyy" value="0.02" />
   <xacro:property name="thigh_izz" value="0.01" />
   <!-- Knee properties -->
-  <xacro:property name="knee_radius" value="0.06" />
+  <xacro:property name="knee_radius" value="0.04" />
   <!-- Shin properties -->
-  <xacro:property name="shin_radius" value="0.06" />
-  <xacro:property name="shin_length" value="0.25" />
-  <xacro:property name="shin_mass" value="1.5" />
+  <xacro:property name="shin_radius" value="0.035" />
+  <xacro:property name="shin_length" value="0.33" />
+  <xacro:property name="shin_mass" value="1.0" />
   <xacro:property name="shin_ixx" value="0.015" />
   <xacro:property name="shin_iyy" value="0.015" />
   <xacro:property name="shin_izz" value="0.008" />
   <!-- Foot properties -->
-  <xacro:property name="foot_length" value="0.4" />
-  <xacro:property name="foot_width" value="0.25" />
-  <xacro:property name="foot_height" value="0.05" />
+  <xacro:property name="foot_length" value="0.2" />
+  <xacro:property name="foot_width" value="0.1" />
+  <xacro:property name="foot_height" value="0.03" />
   <xacro:property name="foot_offset_front" value="0.05" />
-  <xacro:property name="foot_mass" value="0.5" />
-  <xacro:property name="foot_ixx" value="0.002" />
-  <xacro:property name="foot_iyy" value="0.002" />
-  <xacro:property name="foot_izz" value="0.001" />
+  <xacro:property name="foot_mass" value="0.3" />
+  <xacro:property name="foot_ixx" value="0.001" />
+  <xacro:property name="foot_iyy" value="0.001" />
+  <xacro:property name="foot_izz" value="0.0005" />
   <!-- Head properties -->
-  <xacro:property name="head_radius" value="0.15" />
-  <xacro:property name="head_mass" value="0.1" />
-  <xacro:property name="head_ixx" value="0.01" />
-  <xacro:property name="head_iyy" value="0.01" />
-  <xacro:property name="head_izz" value="0.01" />
+  <xacro:property name="head_radius" value="0.1" />
+  <xacro:property name="head_mass" value="0.2" />
+  <xacro:property name="head_ixx" value="0.005" />
+  <xacro:property name="head_iyy" value="0.005" />
+  <xacro:property name="head_izz" value="0.005" />
   <!-- IMU properties -->
-  <xacro:property name="imu_length" value="0.03" />
-  <xacro:property name="imu_width" value="0.05" />
-  <xacro:property name="imu_height" value="0.05" />
+  <xacro:property name="imu_length" value="0.02" />
+  <xacro:property name="imu_width" value="0.03" />
+  <xacro:property name="imu_height" value="0.01" />
   <xacro:property name="imu_mass" value="0.01" />
-  <xacro:property name="imu_ixx" value="0.0001" />
-  <xacro:property name="imu_iyy" value="0.0001" />
-  <xacro:property name="imu_izz" value="0.0001" />
+  <xacro:property name="imu_ixx" value="0.00001" />
+  <xacro:property name="imu_iyy" value="0.00001" />
+  <xacro:property name="imu_izz" value="0.00001" />
   <!-- Materials -->
   <material name="robot_material_1">
-    <color rgba="0.37 0.09 0.09 1"/>
+    <color rgba="0.7 0.7 0.8 1"/>
   </material>
   <material name="robot_material_2">
-    <color rgba="0.37 0.09 1.00 1"/>
+    <color rgba="0.9 0.9 1.0 1"/>
   </material>
+  <!-- altura total -->
+  <xacro:property name="total_height" value="${foot_height + shin_length + thigh_length + body_length + head_radius*2}" />
+  <xacro:property name="base_z" value="${total_height/2}" />
   <!-- Body (main cylinder) -->
   <link name="base_link">
-    <origin xyz="0 0 0"/>
     <visual>
-      <!-- Z: body_length/2 shifts the Z plane from the cylinder's center to its base -->
-      <!-- Z: thigh_length + shin_length + foot_height gives space for the legs -->
-      <origin xyz="0 0 ${body_length/2 + thigh_length + shin_length + foot_height}"/>
+      <origin xyz="0 0 ${base_z - foot_height - shin_length - thigh_length - body_length/2}"/>
       <geometry>
         <cylinder length="${body_length}" radius="${body_radius}"/>
@@ -69,5 +69,5 @@
     </visual>
     <collision>
-      <origin xyz="0 0 ${body_length/2 + thigh_length + shin_length + foot_height}"/>
+      <origin xyz="0 0 ${base_z - foot_height - shin_length - thigh_length - body_length/2}"/>
       <geometry>
         <cylinder length="${body_length}" radius="${body_radius}"/>
@@ -102,14 +102,9 @@
     <parent link="base_link"/>
     <child link="imu_link"/>
-    <!-- Z: Since the body is positioned at 0 0 0, move the joint considering the length of the legs and part of the body -->
-    <!-- Z: Move the IMU foot_height + shin_length + thigh_length, to place it above the legs -->
-    <!-- Z: Move the IMU body_length/3 to place it around the middle of the body -->
-    <!-- X: Move the IMU body_radius to place it at the edge of the body -->
-    <origin xyz="${body_radius} 0 ${foot_height + shin_length + thigh_length + body_length/3 }" rpy="0 0 0"/>
+    <origin xyz="${body_radius} 0 ${body_length/2 }" rpy="0 0 0"/>
   </joint>
   <!-- Head (sphere) -->
   <link name="head_link">
     <visual>
-      <!-- Z: head_radius shifts the Z plane from the heads's center to its base -->
       <origin rpy="0 0 0" xyz="0 0 ${head_radius}"/>
       <geometry>
@@ -133,6 +128,5 @@
     <parent link="base_link"/>
     <child link="head_link"/>
-    <!-- Z: Since the body is positioned at 0 0 0, move the joint up considering the length of the legs and the body -->
-	  <origin xyz="0 0 ${foot_height + shin_length + thigh_length + body_length}"/>
+	  <origin xyz="0 0 ${body_length/2 + head_radius}"/>
   </joint>
   <!-- Leg macro (creates left/right leg: thigh, shin, foot) -->
@@ -141,7 +135,5 @@
     <link name="${prefix}_thigh_link">
       <visual>
-        <!-- Z: thigh_length/2 shifts the Z plane from the thigh's center to its base -->
-        <!-- Z: hip_radius takes the thigh outside of the hip -->
-        <origin rpy="0 0 0" xyz="0 0 ${-thigh_length/2 - hip_radius}"/>
+        <origin rpy="0 0 0" xyz="0 0 ${-thigh_length/2}"/>
         <geometry>
           <cylinder length="${thigh_length}" radius="${thigh_radius}"/>
@@ -150,5 +142,5 @@
       </visual>
       <collision>
-        <origin rpy="0 0 0" xyz="0 0 ${-thigh_length/2 - hip_radius}"/>
+        <origin rpy="0 0 0" xyz="0 0 ${thigh_length/2}"/>
         <geometry>
           <cylinder length="${thigh_length}" radius="${thigh_radius}"/>
@@ -164,18 +156,12 @@
       <parent link="base_link"/>
       <child link="${prefix}_thigh_link"/>
-      <!-- Z: Since the body is positioned at 0 0 0, move the joint up considering the length of the legs -->
-      <!-- Z: Move the joint hip_radius to make it's bottom coincide with the body's bottom -->
-      <!-- Y: Move the joint body_radius to place it at the edge of the body -->
-      <!-- Y: Move the joint hip_radius to take it outside of the body -->
-      <origin xyz="0 ${(body_radius + hip_radius) * reflect} ${thigh_length + shin_length + foot_height + hip_radius}"/>
+      <origin xyz="0 ${body_radius * reflect} ${-body_length/2}"/>
       <axis xyz="0 1 0"/>
-      <limit lower="-1.57" upper="1.57" effort="50" velocity="5"/>
+      <limit lower="-1.0" upper="1.0" effort="100" velocity="8"/>
     </joint>
     <!-- Shin -->
     <link name="${prefix}_shin_link">
       <visual>
-        <!-- Z: shin_length/2 shifts the Z plane from the thigh's center to its base -->
-        <!-- Z: knee_radius takes the thigh outside of the hip -->
-        <origin rpy="0 0 0" xyz="0 0 ${-shin_length/2 - knee_radius}"/>
+        <origin rpy="0 0 0" xyz="0 0 ${-shin_length/2}"/>
         <geometry>
           <cylinder length="${shin_length}" radius="${shin_radius}"/>
@@ -184,5 +170,5 @@
       </visual>
       <collision>
-        <origin rpy="0 0 0" xyz="0 0 ${-shin_length/2 - knee_radius}"/>
+        <origin rpy="0 0 0" xyz="0 0 ${shin_length/2}"/>
         <geometry>
           <cylinder length="${shin_length}" radius="${shin_radius}"/>
@@ -198,17 +184,11 @@
       <parent link="${prefix}_thigh_link"/>
       <child link="${prefix}_shin_link"/>
-      <!-- Z: Move the joint hip_radius + thigh_length to make it's center coincide with the thigh's bottom -->
-      <!-- Z: Move the joint knee_radius to make it's bottom coincide with the thigh's bottom -->
-      <!-- Y: Move the joint thigh_radius to place it at the edge of the thigh -->
-      <!-- Y: Move the joint knee_radius to take it outside of the thigh -->
-      <origin xyz="0 ${(-thigh_radius + -knee_radius) * reflect} ${-hip_radius - thigh_length + knee_radius}"/>
+      <origin xyz="0 0 ${-thigh_length/2}"/>
       <axis xyz="0 1 0"/>
-      <limit lower="0" upper="2.36" effort="40" velocity="5"/>
+      <limit lower="-0.5" upper="2.0" effort="60" velocity="8"/>
     </joint>
     <!-- Foot -->
     <link name="${prefix}_foot_link">
       <visual>
-        <!-- Z: foot_height/2 shifts the Z plane from the foots's center to its top -->
-        <!-- X: foot_offset_front shifts the foot to the front -->
         <origin rpy="0 0 0" xyz="${foot_offset_front} 0 ${-foot_height/2}"/>
         <geometry>
@@ -232,5 +212,4 @@
       <parent link="${prefix}_shin_link"/>
       <child link="${prefix}_foot_link"/>
-      <!-- Z: Move the joint knee_radius + shin_length to make it's center coincide with the shin's bottom -->
       <origin xyz="0 0 ${-knee_radius - shin_length}"/>
     </joint>

Commit message: Arrumar robot_stage1

File: robots/robot_stage1.xacro (robot description, xacro)
@@ -59,8 +59,13 @@
   <xacro:property name="total_height" value="${foot_height + shin_length + thigh_length + body_length + head_radius*2}" />
   <xacro:property name="base_z" value="${total_height/2}" />
+  <xacro:property name="leg_total_length" value="${thigh_length + shin_length + foot_height}" />
+  <!-- body_offset: body_length/2 desloca o posicao Z do centro do cilindro (corpo do robo) para a sua base inferior, assim nao fica metade do corpo enterrado no chao -->
+  <!-- body_offset: leg_total_length da espaco para as pernas, para elas nao ficarem enterradas no chao -->
+  <xacro:property name="body_offset" value="${body_length/2 + leg_total_length}" />
   <!-- Body (main cylinder) -->
   <link name="base_link">
+    <origin xyz="0 0 0"/>
     <visual>
-      <origin xyz="0 0 ${base_z - foot_height - shin_length - thigh_length - body_length/2}"/>
+      <origin xyz="0 0 ${body_offset}"/>
       <geometry>
         <cylinder length="${body_length}" radius="${body_radius}"/>
@@ -69,5 +74,5 @@
     </visual>
     <collision>
-      <origin xyz="0 0 ${base_z - foot_height - shin_length - thigh_length - body_length/2}"/>
+      <origin xyz="0 0 ${body_offset}"/>
       <geometry>
         <cylinder length="${body_length}" radius="${body_radius}"/>
@@ -102,9 +107,12 @@
     <parent link="base_link"/>
     <child link="imu_link"/>
-    <origin xyz="${body_radius} 0 ${body_length/2 }" rpy="0 0 0"/>
+    <!-- Z: Como o corpo principal e posicionado em 0 0 0, body_offset move a IMU para o centro do corpo -->
+    <!-- Z: body_length/4 move a IMU um pouco para baixo, como se estivesse posicionado ela na cintura -->
+    <origin xyz="${body_radius} 0 ${body_offset - body_length/4}" rpy="0 0 0"/>
   </joint>
   <!-- Head (sphere) -->
   <link name="head_link">
     <visual>
+      <!-- Z: head_radius shifts the Z plane from the heads's center to its base -->
       <origin rpy="0 0 0" xyz="0 0 ${head_radius}"/>
       <geometry>
@@ -128,5 +136,7 @@
     <parent link="base_link"/>
     <child link="head_link"/>
-	  <origin xyz="0 0 ${body_length/2 + head_radius}"/>
+    <!-- Z: Como o corpo principal e posicionado em 0 0 0, body_offset move a joint para o centro do corpo -->
+    <!-- Z: body_length/2 move a joint para o topo do corpo -->
+	  <origin xyz="0 0 ${body_offset + body_length/2}"/>
   </joint>
   <!-- Leg macro (creates left/right leg: thigh, shin, foot) -->
@@ -135,5 +145,7 @@
     <link name="${prefix}_thigh_link">
       <visual>
-        <origin rpy="0 0 0" xyz="0 0 ${-thigh_length/2}"/>
+        <!-- Z: thigh_length/2 desloca a posicao Z do centro do cilindro para a sua base inferior -->
+        <!-- Z: hip_radius desloca a coxa para fora do quadril -->
+        <origin rpy="0 0 0" xyz="0 0 ${-thigh_length/2 - hip_radius}"/>
         <geometry>
           <cylinder length="${thigh_length}" radius="${thigh_radius}"/>
@@ -142,5 +154,5 @@
       </visual>
       <collision>
-        <origin rpy="0 0 0" xyz="0 0 ${thigh_length/2}"/>
+        <origin rpy="0 0 0" xyz="0 0 ${-thigh_length/2 - hip_radius}"/>
         <geometry>
           <cylinder length="${thigh_length}" radius="${thigh_radius}"/>
@@ -156,12 +168,19 @@
       <parent link="base_link"/>
       <child link="${prefix}_thigh_link"/>
-      <origin xyz="0 ${body_radius * reflect} ${-body_length/2}"/>
+      <!-- Z: Como o corpo principal e posicionado em 0 0 0, body_offset move a joint para o centro do corpo -->
+      <!-- Z: body_length/2 move a joint para a base inferior do corpo -->
+      <!-- Z: hip_radius faz a base inferior do quadrilcoincidir com a base inferior do corpo -->
+      <!-- Y: body_radius posiciona a joint na borda do corpo -->
+      <!-- Y: hip_radius tira o quadrilde dentro do corpo, caso contrario metade do quadrilficaria dentro do corpo -->
+      <origin xyz="0 ${(body_radius + hip_radius) * reflect} ${body_offset - body_length/2 + hip_radius}"/>
       <axis xyz="0 1 0"/>
-      <limit lower="-1.0" upper="1.0" effort="100" velocity="8"/>
+      <limit lower="-1.57" upper="1.57" effort="50" velocity="5"/>
     </joint>
     <!-- Shin -->
     <link name="${prefix}_shin_link">
       <visual>
-        <origin rpy="0 0 0" xyz="0 0 ${-shin_length/2}"/>
+        <!-- Z: shin_length/2 desloca a posicao Z do centro da coxa para a sua base inferior -->
+        <!-- Z: knee_radius tira a coxa de dentro do quadril-->
+        <origin rpy="0 0 0" xyz="0 0 ${-shin_length/2 - knee_radius}"/>
         <geometry>
           <cylinder length="${shin_length}" radius="${shin_radius}"/>
@@ -170,5 +189,5 @@
       </visual>
       <collision>
-        <origin rpy="0 0 0" xyz="0 0 ${shin_length/2}"/>
+        <origin rpy="0 0 0" xyz="0 0 ${-shin_length/2 - knee_radius}"/>
         <geometry>
           <cylinder length="${shin_length}" radius="${shin_radius}"/>
@@ -184,11 +203,17 @@
       <parent link="${prefix}_thigh_link"/>
       <child link="${prefix}_shin_link"/>
-      <origin xyz="0 0 ${-thigh_length/2}"/>
+      <!-- Z: hip_radius + thigh_length faz o centro da cenela coincidir com a base inferior da coxa -->
+      <!-- Z: knee_radius faz a base inferior da cenela coincidir com a base inferior da coxa -->
+      <!-- Y: thigh_radius posiciona o centro da cenela na borda da coxa -->
+      <!-- Y: knee_radius coloca a cenela para fora da coxa -->
+      <origin xyz="0 ${(-thigh_radius + -knee_radius) * reflect} ${-hip_radius - thigh_length + knee_radius}"/>
       <axis xyz="0 1 0"/>
-      <limit lower="-0.5" upper="2.0" effort="60" velocity="8"/>
+      <limit lower="0" upper="2.36" effort="40" velocity="5"/>
     </joint>
     <!-- Foot -->
     <link name="${prefix}_foot_link">
       <visual>
+        <!-- Z: foot_height/2 desloca a posicao Z do centro do pe para o seu topo -->
+        <!-- X: foot_offset_front desloca o pe um pouco para frente, para parecer um pe normal em que ele fica mais para frente do que para tras -->
         <origin rpy="0 0 0" xyz="${foot_offset_front} 0 ${-foot_height/2}"/>
         <geometry>
@@ -212,4 +237,5 @@
       <parent link="${prefix}_shin_link"/>
       <child link="${prefix}_foot_link"/>
+      <!-- Z: knee_radius + shin_length faz o centro do pe coincidir com o centro da cenela -->
       <origin xyz="0 0 ${-knee_radius - shin_length}"/>
     </joint>

Commit message: Remover propriedades nao usadas

File: robots/robot_stage1.xacro (robot description, xacro)
@@ -57,6 +57,4 @@
   </material>
   <!-- altura total -->
-  <xacro:property name="total_height" value="${foot_height + shin_length + thigh_length + body_length + head_radius*2}" />
-  <xacro:property name="base_z" value="${total_height/2}" />
   <xacro:property name="leg_total_length" value="${thigh_length + shin_length + foot_height}" />
   <!-- body_offset: body_length/2 desloca o posicao Z do centro do cilindro (corpo do robo) para a sua base inferior, assim nao fica metade do corpo enterrado no chao -->

Commit message: Corrigir collision do pé do robô 1

File: robots/robot_stage1.xacro (robot description, xacro)
@@ -222,5 +222,5 @@
       </visual>
       <collision>
-        <origin rpy="0 0 0" xyz="0 0 ${-foot_height/2}"/>
+        <origin rpy="0 0 0" xyz="${foot_offset_front} 0 ${-foot_height/2}"/>
         <geometry>
           <box size="${foot_length} ${foot_width} ${foot_height}"/>
