Commit message: Adicionar articulação ao tornozelo

File: robots/robot_stage4.xacro (robot description, xacro)
@@ -288,5 +288,5 @@
     </link>
     <!-- Ankle joint: shin to ankle ball -->
-    <joint name="${prefix}_shin_to_ankle_ball" type="fixed">
+    <joint name="${prefix}_shin_to_ankle_ball" type="revolute">
       <parent link="${prefix}_shin_link"/>
       <child link="${prefix}_ankle_ball_link"/>
@@ -295,4 +295,7 @@
       <!-- Z: Diminuir ankle_radius faz o topo da esfera/articulacao do tornozelo coincidir com a base inferior da canela -->
       <origin xyz="0 0 ${-knee_radius - shin_length - ankle_radius}"/>
+      <axis xyz="0 1 0"/> <!-- Movimento frontal -->
+      <limit lower="${-30 * deg_to_rad}" upper="${75 * deg_to_rad}" effort="1000" velocity="5"/>
+      <dynamics damping="${joint_dumping}" friction="${joint_friction}"/>
     </joint>
     <!-- Ankle Ball -->
@@ -321,6 +324,6 @@
       <child link="${prefix}_foot_link"/>
       <origin xyz="0 0 0"/>
-      <axis xyz="0 1 0"/>
-      <limit lower="${-30 * deg_to_rad}" upper="${75 * deg_to_rad}" effort="1000" velocity="5"/>
+      <axis xyz="1 0 0"/> <!-- Movimento lateral -->
+      <limit lower="${-30 * deg_to_rad}" upper="${30 * deg_to_rad}" effort="1000" velocity="5"/>
       <dynamics damping="${joint_dumping}" friction="${joint_friction}"/>
     </joint>

Commit message: Ajustar limites de articulações

File: robots/robot_stage4.xacro (robot description, xacro)
@@ -171,5 +171,5 @@
       <origin xyz="0 ${(body_radius + hip_radius) * reflect} ${body_offset - body_length/2}"/>
       <axis xyz="0 1 0"/> <!-- Movimento frontal -->
-      <limit lower="${-90 * deg_to_rad}" upper="${90 * deg_to_rad}" effort="1000" velocity="5"/>
+      <limit lower="${-75 * deg_to_rad}" upper="${60 * deg_to_rad}" effort="1000" velocity="5"/>
       <dynamics damping="${joint_dumping}" friction="${joint_friction}"/>
     </joint>
@@ -261,5 +261,5 @@
       <origin xyz="0 0 0"/>
       <axis xyz="0 1 0"/>
-      <limit lower="${0 * deg_to_rad}" upper="${135 * deg_to_rad}" effort="1000" velocity="5"/>
+      <limit lower="${0 * deg_to_rad}" upper="${90 * deg_to_rad}" effort="1000" velocity="5"/>
       <dynamics damping="${joint_dumping}" friction="${joint_friction}"/>
     </joint>

Commit message: Diminuir abertura máxima das pernas do robô 4

File: robots/robot_stage4.xacro (robot description, xacro)
@@ -199,5 +199,5 @@
       <origin xyz="0 0 0"/>
       <axis xyz="1 0 0"/> <!-- Movimento lateral -->
-      <limit lower="${-30 * deg_to_rad}" upper="${30 * deg_to_rad}" effort="1000" velocity="5"/>
+      <limit lower="${-20 * deg_to_rad}" upper="${20 * deg_to_rad}" effort="1000" velocity="5"/>
       <dynamics damping="${joint_damping}" friction="${joint_friction}"/>
     </joint>

Commit message: Corrigir inércia do robô

File: robots/robot_stage4.xacro (robot description, xacro)
@@ -5,39 +5,45 @@
   <xacro:property name="body_length" value="0.3" />
   <xacro:property name="body_mass" value="5.0" />
-  <xacro:property name="body_ixx" value="0.1" />
-  <xacro:property name="body_iyy" value="0.1" />
-  <xacro:property name="body_izz" value="0.05" />
+  <!-- Inertia for solid cylinder (axis z): Ixx = Iyy = (1/12)*m*(3*r^2+h^2); Izz = (1/2)*m*r^2 -->
+  <xacro:property name="body_ixx" value="${(1.0/12.0) * body_mass * (3 * body_radius * body_radius + body_length * body_length)}" />
+  <xacro:property name="body_iyy" value="${(1.0/12.0) * body_mass * (3 * body_radius * body_radius + body_length * body_length)}" />
+  <xacro:property name="body_izz" value="${0.5 * body_mass * body_radius * body_radius}" />
   <!-- Hip properties -->
   <xacro:property name="hip_radius" value="0.05" />
   <xacro:property name="hip_mass" value="0.5" />
-  <xacro:property name="hip_ixx" value="0.01" />
-  <xacro:property name="hip_iyy" value="0.01" />
-  <xacro:property name="hip_izz" value="0.01" />
+  <!-- Inertia for solid sphere: Ixx = Iyy = Izz = (2/5)*m*r^2 -->
+  <xacro:property name="hip_ixx" value="${0.4 * hip_mass * hip_radius * hip_radius}" />
+  <xacro:property name="hip_iyy" value="${0.4 * hip_mass * hip_radius * hip_radius}" />
+  <xacro:property name="hip_izz" value="${0.4 * hip_mass * hip_radius * hip_radius}" />
   <!-- Thigh properties -->
   <xacro:property name="thigh_radius" value="0.04" />
   <xacro:property name="thigh_length" value="0.35" />
   <xacro:property name="thigh_mass" value="1.5" />
-  <xacro:property name="thigh_ixx" value="0.02" />
-  <xacro:property name="thigh_iyy" value="0.02" />
-  <xacro:property name="thigh_izz" value="0.01" />
+  <!-- Inertia for solid cylinder (axis z): Ixx = Iyy = (1/12)*m*(3*r^2+h^2); Izz = (1/2)*m*r^2 -->
+  <xacro:property name="thigh_ixx" value="${(1.0/12.0) * thigh_mass * (3 * thigh_radius * thigh_radius + thigh_length * thigh_length)}" />
+  <xacro:property name="thigh_iyy" value="${(1.0/12.0) * thigh_mass * (3 * thigh_radius * thigh_radius + thigh_length * thigh_length)}" />
+  <xacro:property name="thigh_izz" value="${0.5 * thigh_mass * thigh_radius * thigh_radius}" />
   <!-- Knee properties -->
   <xacro:property name="knee_radius" value="0.04" />
   <xacro:property name="knee_mass" value="0.5" />
-  <xacro:property name="knee_ixx" value="0.01" />
-  <xacro:property name="knee_iyy" value="0.01" />
-  <xacro:property name="knee_izz" value="0.01" />
+  <!-- Inertia for solid sphere: Ixx = Iyy = Izz = (2/5)*m*r^2 -->
+  <xacro:property name="knee_ixx" value="${0.4 * knee_mass * knee_radius * knee_radius}" />
+  <xacro:property name="knee_iyy" value="${0.4 * knee_mass * knee_radius * knee_radius}" />
+  <xacro:property name="knee_izz" value="${0.4 * knee_mass * knee_radius * knee_radius}" />
   <!-- Shin properties -->
   <xacro:property name="shin_radius" value="0.035" />
   <xacro:property name="shin_length" value="0.30" />
   <xacro:property name="shin_mass" value="1.5" />
-  <xacro:property name="shin_ixx" value="0.015" />
-  <xacro:property name="shin_iyy" value="0.015" />
-  <xacro:property name="shin_izz" value="0.008" />
+  <!-- Inertia for solid cylinder (axis z): Ixx = Iyy = (1/12)*m*(3*r^2+h^2); Izz = (1/2)*m*r^2 -->
+  <xacro:property name="shin_ixx" value="${(1.0/12.0) * shin_mass * (3 * shin_radius * shin_radius + shin_length * shin_length)}" />
+  <xacro:property name="shin_iyy" value="${(1.0/12.0) * shin_mass * (3 * shin_radius * shin_radius + shin_length * shin_length)}" />
+  <xacro:property name="shin_izz" value="${0.5 * shin_mass * shin_radius * shin_radius}" />
   <!-- Ankle properties -->
   <xacro:property name="ankle_radius" value="0.03" />
   <xacro:property name="ankle_mass" value="0.5" />
-  <xacro:property name="ankle_ixx" value="0.01" />
-  <xacro:property name="ankle_iyy" value="0.01" />
-  <xacro:property name="ankle_izz" value="0.01" />
+  <!-- Inertia for solid sphere: Ixx = Iyy = Izz = (2/5)*m*r^2 -->
+  <xacro:property name="ankle_ixx" value="${0.4 * ankle_mass * ankle_radius * ankle_radius}" />
+  <xacro:property name="ankle_iyy" value="${0.4 * ankle_mass * ankle_radius * ankle_radius}" />
+  <xacro:property name="ankle_izz" value="${0.4 * ankle_mass * ankle_radius * ankle_radius}" />
   <!-- Foot properties -->
   <xacro:property name="foot_length" value="0.35" />
@@ -46,13 +52,15 @@
   <xacro:property name="foot_offset_front" value="0.1" />
   <xacro:property name="foot_mass" value="0.5" />
-  <xacro:property name="foot_ixx" value="0.001" />
-  <xacro:property name="foot_iyy" value="0.001" />
-  <xacro:property name="foot_izz" value="0.0005" />
+  <!-- Inertia for box (length, width, height): Ixx = (1/12)*m*(w^2+h^2); Iyy = (1/12)*m*(l^2+h^2); Izz = (1/12)*m*(l^2+w^2) -->
+  <xacro:property name="foot_ixx" value="${(1.0/12.0) * foot_mass * (foot_width * foot_width + foot_height * foot_height)}" />
+  <xacro:property name="foot_iyy" value="${(1.0/12.0) * foot_mass * (foot_length * foot_length + foot_height * foot_height)}" />
+  <xacro:property name="foot_izz" value="${(1.0/12.0) * foot_mass * (foot_length * foot_length + foot_width * foot_width)}" />
   <!-- Head properties -->
   <xacro:property name="head_radius" value="0.1" />
   <xacro:property name="head_mass" value="1.0" />
-  <xacro:property name="head_ixx" value="0.005" />
-  <xacro:property name="head_iyy" value="0.005" />
-  <xacro:property name="head_izz" value="0.005" />
+  <!-- Inertia for solid sphere: Ixx = Iyy = Izz = (2/5)*m*r^2 -->
+  <xacro:property name="head_ixx" value="${0.4 * head_mass * head_radius * head_radius}" />
+  <xacro:property name="head_iyy" value="${0.4 * head_mass * head_radius * head_radius}" />
+  <xacro:property name="head_izz" value="${0.4 * head_mass * head_radius * head_radius}" />
   <!-- IMU properties -->
   <xacro:property name="imu_length" value="0.02" />
@@ -60,7 +68,8 @@
   <xacro:property name="imu_height" value="0.01" />
   <xacro:property name="imu_mass" value="0.01" />
-  <xacro:property name="imu_ixx" value="0.00001" />
-  <xacro:property name="imu_iyy" value="0.00001" />
-  <xacro:property name="imu_izz" value="0.00001" />
+  <!-- Inertia for box (length, width, height): Ixx = (1/12)*m*(w^2+h^2); Iyy = (1/12)*m*(l^2+h^2); Izz = (1/12)*m*(l^2+w^2) -->
+  <xacro:property name="imu_ixx" value="${(1.0/12.0) * imu_mass * (imu_width * imu_width + imu_height * imu_height)}" />
+  <xacro:property name="imu_iyy" value="${(1.0/12.0) * imu_mass * (imu_length * imu_length + imu_height * imu_height)}" />
+  <xacro:property name="imu_izz" value="${(1.0/12.0) * imu_mass * (imu_length * imu_length + imu_width * imu_width)}" />
   <!-- Controle -->
   <xacro:property name="joint_damping" value="0.2" />
