Commit message: Corrigir xacro

File: robots/robot_s4_realista.xacro (robot description, xacro)
@@ -50,5 +50,5 @@
   <xacro:property name="foot_width" value="0.10" />
   <xacro:property name="foot_height" value="0.05" />
-  <xacro:property name="foot_offset_front" value="0.15 />
+  <xacro:property name="foot_offset_front" value="0.15" />
   <xacro:property name="foot_mass" value="2.1" />
   <!-- Inertia for box (length, width, height): Ixx = (1/12)*m*(w^2+h^2); Iyy = (1/12)*m*(l^2+h^2); Izz = (1/12)*m*(l^2+w^2) -->
