Commit message: estou tentando o 08 e 010

File: robots/robot_stage4.010.xacro (robot description, xacro)
@@ -3,5 +3,5 @@
   <!-- Body properties -->
   <xacro:property name="body_radius" value="0.15" />
-  <xacro:property name="body_length" value="0.3" />
+  <xacro:property name="body_length" value="0.5" />
   <xacro:property name="body_mass" value="5.0" />
   <!-- Inertia for solid cylinder (axis z): Ixx = Iyy = (1/12)*m*(3*r^2+h^2); Izz = (1/2)*m*r^2 -->
@@ -19,5 +19,5 @@
   <xacro:property name="thigh_radius" value="0.075" />
   <xacro:property name="thigh_length" value="0.40" />
-  <xacro:property name="thigh_mass" value="18.5" />
+  <xacro:property name="thigh_mass" value="1.5" />
   <!-- Inertia for solid cylinder (axis z): Ixx = Iyy = (1/12)*m*(3*r^2+h^2); Izz = (1/2)*m*r^2 -->
   <xacro:property name="thigh_ixx" value="${(1.0/12.0) * thigh_mass * (3 * thigh_radius * thigh_radius + thigh_length * thigh_length)}" />
@@ -34,5 +34,5 @@
   <xacro:property name="shin_radius" value="0.06" />
   <xacro:property name="shin_length" value="0.43" />
-  <xacro:property name="shin_mass" value="7.6" />
+  <xacro:property name="shin_mass" value="1.5" />
   <!-- Inertia for solid cylinder (axis z): Ixx = Iyy = (1/12)*m*(3*r^2+h^2); Izz = (1/2)*m*r^2 -->
   <xacro:property name="shin_ixx" value="${(1.0/12.0) * shin_mass * (3 * shin_radius * shin_radius + shin_length * shin_length)}" />
@@ -51,5 +51,5 @@
   <xacro:property name="foot_height" value="0.05" />
   <xacro:property name="foot_offset_front" value="0.1" />
-  <xacro:property name="foot_mass" value="2.1" />
+  <xacro:property name="foot_mass" value="0.5" />
   <!-- Inertia for box (length, width, height): Ixx = (1/12)*m*(w^2+h^2); Iyy = (1/12)*m*(l^2+h^2); Izz = (1/12)*m*(l^2+w^2) -->
   <xacro:property name="foot_ixx" value="${(1.0/12.0) * foot_mass * (foot_width * foot_width + foot_height * foot_height)}" />

File: robots/robot_stage4.08.xacro (robot description, xacro)
@@ -181,6 +181,6 @@
       <!-- Y: hip_radius tira a esfera/articulacao de dentro do corpo, caso contrario metade da esfera/articulacao ficaria dentro do corpo -->
       <origin xyz="0 ${(body_radius + hip_radius) * reflect} ${body_offset - body_length/2}"/>
-      <axis xyz="0 1 0"/> <!-- Movimento frontal -->
-      <limit lower="${-75 * deg_to_rad}" upper="${60 * deg_to_rad}" effort="1000" velocity="5"/>
+      <axis xyz="0 1 0"/>
+      <limit lower="${-45 * deg_to_rad}" upper="${45 * deg_to_rad}" effort="${joint_effort}" velocity="${joint_velocity}"/>
       <dynamics damping="${joint_damping}" friction="${joint_friction}"/>
     </joint>
@@ -211,5 +211,5 @@
       <origin xyz="0 0 0"/>
       <axis xyz="1 0 0"/> <!-- Movimento lateral -->
-      <limit lower="${-20 * deg_to_rad}" upper="${20 * deg_to_rad}" effort="1000" velocity="5"/>
+      <limit lower="${-25 * deg_to_rad}" upper="${25 * deg_to_rad}" effort="${joint_effort}" velocity="${joint_velocity}"/>
       <dynamics damping="${joint_damping}" friction="${joint_friction}"/>
     </joint>
@@ -272,5 +272,5 @@
       <origin xyz="0 0 0"/>
       <axis xyz="0 1 0"/>
-      <limit lower="${0 * deg_to_rad}" upper="${90 * deg_to_rad}" effort="1000" velocity="5"/>
+      <limit lower="${0 * deg_to_rad}" upper="${90 * deg_to_rad}" effort="${joint_effort}" velocity="${joint_velocity}"/>
       <dynamics damping="${joint_damping}" friction="${joint_friction}"/>
     </joint>
@@ -307,5 +307,5 @@
       <origin xyz="0 0 ${-knee_radius - shin_length - ankle_radius}"/>
       <axis xyz="0 1 0"/> <!-- Movimento frontal -->
-      <limit lower="${-30 * deg_to_rad}" upper="${75 * deg_to_rad}" effort="1000" velocity="5"/>
+      <limit lower="${-20 * deg_to_rad}" upper="${20 * deg_to_rad}" effort="${joint_effort}" velocity="${joint_velocity}"/>
       <dynamics damping="${joint_damping}" friction="${joint_friction}"/>
     </joint>
@@ -336,5 +336,5 @@
       <origin xyz="0 0 0"/>
       <axis xyz="1 0 0"/> <!-- Movimento lateral -->
-      <limit lower="${-30 * deg_to_rad}" upper="${30 * deg_to_rad}" effort="1000" velocity="5"/>
+      <limit lower="${-10 * deg_to_rad}" upper="${10 * deg_to_rad}" effort="${joint_effort}" velocity="${joint_velocity}"/>
       <dynamics damping="${joint_damping}" friction="${joint_friction}"/>
     </joint>

File: robots/robot_stage4.09.xacro (robot description, xacro)
@@ -181,6 +181,6 @@
       <!-- Y: hip_radius tira a esfera/articulacao de dentro do corpo, caso contrario metade da esfera/articulacao ficaria dentro do corpo -->
       <origin xyz="0 ${(body_radius + hip_radius) * reflect} ${body_offset - body_length/2}"/>
-      <axis xyz="0 1 0"/> <!-- Movimento frontal -->
-      <limit lower="${-75 * deg_to_rad}" upper="${60 * deg_to_rad}" effort="1000" velocity="5"/>
+      <axis xyz="0 1 0"/>
+      <limit lower="${-45 * deg_to_rad}" upper="${45 * deg_to_rad}" effort="${joint_effort}" velocity="${joint_velocity}"/>
       <dynamics damping="${joint_damping}" friction="${joint_friction}"/>
     </joint>
@@ -211,5 +211,5 @@
       <origin xyz="0 0 0"/>
       <axis xyz="1 0 0"/> <!-- Movimento lateral -->
-      <limit lower="${-20 * deg_to_rad}" upper="${20 * deg_to_rad}" effort="1000" velocity="5"/>
+      <limit lower="${-25 * deg_to_rad}" upper="${25 * deg_to_rad}" effort="${joint_effort}" velocity="${joint_velocity}"/>
       <dynamics damping="${joint_damping}" friction="${joint_friction}"/>
     </joint>
@@ -272,5 +272,5 @@
       <origin xyz="0 0 0"/>
       <axis xyz="0 1 0"/>
-      <limit lower="${0 * deg_to_rad}" upper="${90 * deg_to_rad}" effort="1000" velocity="5"/>
+      <limit lower="${0 * deg_to_rad}" upper="${90 * deg_to_rad}" effort="${joint_effort}" velocity="${joint_velocity}"/>
       <dynamics damping="${joint_damping}" friction="${joint_friction}"/>
     </joint>
@@ -307,5 +307,5 @@
       <origin xyz="0 0 ${-knee_radius - shin_length - ankle_radius}"/>
       <axis xyz="0 1 0"/> <!-- Movimento frontal -->
-      <limit lower="${-30 * deg_to_rad}" upper="${75 * deg_to_rad}" effort="1000" velocity="5"/>
+      <limit lower="${-20 * deg_to_rad}" upper="${20 * deg_to_rad}" effort="${joint_effort}" velocity="${joint_velocity}"/>
       <dynamics damping="${joint_damping}" friction="${joint_friction}"/>
     </joint>
@@ -336,5 +336,5 @@
       <origin xyz="0 0 0"/>
       <axis xyz="1 0 0"/> <!-- Movimento lateral -->
-      <limit lower="${-30 * deg_to_rad}" upper="${30 * deg_to_rad}" effort="1000" velocity="5"/>
+      <limit lower="${-10 * deg_to_rad}" upper="${10 * deg_to_rad}" effort="${joint_effort}" velocity="${joint_velocity}"/>
       <dynamics damping="${joint_damping}" friction="${joint_friction}"/>
     </joint>
