Commit message: Ajustar 4b: body_length, hip_mass

File: robots/robot_stage4b.xacro (robot description, xacro)
@@ -3,5 +3,5 @@
   <!-- Body properties -->
   <xacro:property name="body_radius" value="0.15" />
-  <xacro:property name="body_length" value="0.3" />
+  <xacro:property name="body_length" value="0.5" />
   <xacro:property name="body_mass" value="5.0" />
   <!-- Inertia for solid cylinder (axis z): Ixx = Iyy = (1/12)*m*(3*r^2+h^2); Izz = (1/2)*m*r^2 -->
@@ -11,5 +11,5 @@
   <!-- Hip properties -->
   <xacro:property name="hip_radius" value="0.05" />
-  <xacro:property name="hip_mass" value="0.5" />
+  <xacro:property name="hip_mass" value="0.0" />
   <!-- Inertia for solid sphere: Ixx = Iyy = Izz = (2/5)*m*r^2 -->
   <xacro:property name="hip_ixx" value="${0.4 * hip_mass * hip_radius * hip_radius}" />

Commit message: Peso do tronco, torque e dimensões da coxa

File: robots/robot_stage4b.xacro (robot description, xacro)
@@ -4,5 +4,5 @@
   <xacro:property name="body_radius" value="0.15" />
   <xacro:property name="body_length" value="0.5" />
-  <xacro:property name="body_mass" value="5.0" />
+  <xacro:property name="body_mass" value="20.0" />
   <!-- Inertia for solid cylinder (axis z): Ixx = Iyy = (1/12)*m*(3*r^2+h^2); Izz = (1/2)*m*r^2 -->
   <xacro:property name="body_ixx" value="${(1.0/12.0) * body_mass * (3 * body_radius * body_radius + body_length * body_length)}" />
@@ -17,6 +17,6 @@
   <xacro:property name="hip_izz" value="${0.4 * hip_mass * hip_radius * hip_radius}" />
   <!-- Thigh properties -->
-  <xacro:property name="thigh_radius" value="0.04" />
-  <xacro:property name="thigh_length" value="0.35" />
+  <xacro:property name="thigh_radius" value="0.075" />
+  <xacro:property name="thigh_length" value="0.3" />   <!-- 0.4 - hip_radius - knee_radius -->
   <xacro:property name="thigh_mass" value="1.5" />
   <!-- Inertia for solid cylinder (axis z): Ixx = Iyy = (1/12)*m*(3*r^2+h^2); Izz = (1/2)*m*r^2 -->

Commit message: Ajustar 4b: thigh_mass

File: robots/robot_stage4b.xacro (robot description, xacro)
@@ -19,5 +19,5 @@
   <xacro:property name="thigh_radius" value="0.075" />
   <xacro:property name="thigh_length" value="0.3" />   <!-- 0.4 - hip_radius - knee_radius -->
-  <xacro:property name="thigh_mass" value="1.5" />
+  <xacro:property name="thigh_mass" value="10.5" />
   <!-- Inertia for solid cylinder (axis z): Ixx = Iyy = (1/12)*m*(3*r^2+h^2); Izz = (1/2)*m*r^2 -->
   <xacro:property name="thigh_ixx" value="${(1.0/12.0) * thigh_mass * (3 * thigh_radius * thigh_radius + thigh_length * thigh_length)}" />

Commit message: Ajustar 4b:  knee, ankle, gait_step_size

File: robots/robot_stage4b.xacro (robot description, xacro)
@@ -25,6 +25,6 @@
   <xacro:property name="thigh_izz" value="${0.5 * thigh_mass * thigh_radius * thigh_radius}" />
   <!-- Knee properties -->
-  <xacro:property name="knee_radius" value="0.04" />
-  <xacro:property name="knee_mass" value="0.5" />
+  <xacro:property name="knee_radius" value="0.05" />
+  <xacro:property name="knee_mass" value="0.0" />
   <!-- Inertia for solid sphere: Ixx = Iyy = Izz = (2/5)*m*r^2 -->
   <xacro:property name="knee_ixx" value="${0.4 * knee_mass * knee_radius * knee_radius}" />
@@ -41,5 +41,5 @@
   <!-- Ankle properties -->
   <xacro:property name="ankle_radius" value="0.03" />
-  <xacro:property name="ankle_mass" value="0.5" />
+  <xacro:property name="ankle_mass" value="0.0" />
   <!-- Inertia for solid sphere: Ixx = Iyy = Izz = (2/5)*m*r^2 -->
   <xacro:property name="ankle_ixx" value="${0.4 * ankle_mass * ankle_radius * ankle_radius}" />

Commit message: Ajustar 4b: head

File: robots/robot_stage4b.xacro (robot description, xacro)
@@ -57,6 +57,6 @@
   <xacro:property name="foot_izz" value="${(1.0/12.0) * foot_mass * (foot_length * foot_length + foot_width * foot_width)}" />
   <!-- Head properties -->
-  <xacro:property name="head_radius" value="0.1" />
-  <xacro:property name="head_mass" value="1.0" />
+  <xacro:property name="head_radius" value="0.09" />
+  <xacro:property name="head_mass" value="4.5" />
   <!-- Inertia for solid sphere: Ixx = Iyy = Izz = (2/5)*m*r^2 -->
   <xacro:property name="head_ixx" value="${0.4 * head_mass * head_radius * head_radius}" />

Commit message: Ajustar 4b: body_mass, shin

File: robots/robot_stage4b.xacro (robot description, xacro)
@@ -4,5 +4,5 @@
   <xacro:property name="body_radius" value="0.15" />
   <xacro:property name="body_length" value="0.5" />
-  <xacro:property name="body_mass" value="20.0" />
+  <xacro:property name="body_mass" value="35.1" />
   <!-- Inertia for solid cylinder (axis z): Ixx = Iyy = (1/12)*m*(3*r^2+h^2); Izz = (1/2)*m*r^2 -->
   <xacro:property name="body_ixx" value="${(1.0/12.0) * body_mass * (3 * body_radius * body_radius + body_length * body_length)}" />
@@ -32,7 +32,7 @@
   <xacro:property name="knee_izz" value="${0.4 * knee_mass * knee_radius * knee_radius}" />
   <!-- Shin properties -->
-  <xacro:property name="shin_radius" value="0.035" />
-  <xacro:property name="shin_length" value="0.30" />
-  <xacro:property name="shin_mass" value="1.5" />
+  <xacro:property name="shin_radius" value="0.06" />
+  <xacro:property name="shin_length" value="0.32" />   <!-- 0.43 - knee_radius - 2 * ankle_radius -->
+  <xacro:property name="shin_mass" value="7.6" />
   <!-- Inertia for solid cylinder (axis z): Ixx = Iyy = (1/12)*m*(3*r^2+h^2); Izz = (1/2)*m*r^2 -->
   <xacro:property name="shin_ixx" value="${(1.0/12.0) * shin_mass * (3 * shin_radius * shin_radius + shin_length * shin_length)}" />

Commit message: Ajustar 4b: neck

File: robots/robot_stage4b.xacro (robot description, xacro)
@@ -9,4 +9,11 @@
   <xacro:property name="body_iyy" value="${(1.0/12.0) * body_mass * (3 * body_radius * body_radius + body_length * body_length)}" />
   <xacro:property name="body_izz" value="${0.5 * body_mass * body_radius * body_radius}" />
+  <!-- Neck properties -->
+  <xacro:property name="neck_radius" value="0.06" />
+  <xacro:property name="neck_length" value="0.10" />
+  <xacro:property name="neck_mass" value="1.0" />
+  <xacro:property name="neck_ixx" value="${(1.0/12.0) * neck_mass * (3 * neck_radius * neck_radius + neck_length * neck_length)}" />
+  <xacro:property name="neck_iyy" value="${(1.0/12.0) * neck_mass * (3 * neck_radius * neck_radius + neck_length * neck_length)}" />
+  <xacro:property name="neck_izz" value="${0.5 * neck_mass * neck_radius * neck_radius}" />
   <!-- Hip properties -->
   <xacro:property name="hip_radius" value="0.05" />
@@ -137,4 +144,30 @@
     <origin xyz="${body_radius} 0 ${body_offset - body_length/4}" rpy="0 0 0"/>
   </joint>
+  <!-- Neck -->
+  <link name="neck_link">
+    <visual>
+      <origin xyz="0 0 ${neck_length/2}" rpy="0 0 0"/>
+      <geometry>
+        <cylinder length="${neck_length}" radius="${neck_radius}"/>
+      </geometry>
+      <material name="robot_material_2"/>
+    </visual>
+    <collision>
+      <origin xyz="0 0 ${neck_length/2}" rpy="0 0 0"/>
+      <geometry>
+        <cylinder length="${neck_length}" radius="${neck_radius}"/>
+      </geometry>
+    </collision>
+    <inertial>
+      <mass value="${neck_mass}"/>
+      <inertia ixx="${neck_ixx}" ixy="0.0" ixz="0.0" iyy="${neck_iyy}" iyz="0.0" izz="${neck_izz}"/>
+    </inertial>
+  </link>
+  <!-- Neck joint: body to neck -->
+  <joint name="base_to_neck" type="fixed">
+    <parent link="base_link"/>
+    <child link="neck_link"/>
+    <origin xyz="0 0 ${body_offset + body_length/2}"/>
+  </joint>
   <!-- Head (sphere) -->
   <link name="head_link">
@@ -159,11 +192,11 @@
     </inertial>
   </link>
-  <!-- Head joint: body to head -->
-  <joint name="base_to_head" type="fixed">
-    <parent link="base_link"/>
+  <!-- Head joint: neck to head -->
+  <joint name="neck_to_head" type="fixed">
+    <parent link="neck_link"/>
     <child link="head_link"/>
     <!-- Z: Como o corpo principal e posicionado em 0 0 0, body_offset move a joint para o centro do corpo -->
     <!-- Z: body_length/2 move a joint para o topo do corpo -->
-	  <origin xyz="0 0 ${body_offset + body_length/2}"/>
+	  <origin xyz="0 0 ${neck_length}"/>
   </joint>
   <!-- Leg macro (creates left/right leg: thigh, shin, foot) -->

Commit message: Ajustar 4b: thigh_mass, max_motor_torque

File: robots/robot_stage4b.xacro (robot description, xacro)
@@ -26,5 +26,5 @@
   <xacro:property name="thigh_radius" value="0.075" />
   <xacro:property name="thigh_length" value="0.3" />   <!-- 0.4 - hip_radius - knee_radius -->
-  <xacro:property name="thigh_mass" value="10.5" />
+  <xacro:property name="thigh_mass" value="18.5" />
   <!-- Inertia for solid cylinder (axis z): Ixx = Iyy = (1/12)*m*(3*r^2+h^2); Izz = (1/2)*m*r^2 -->
   <xacro:property name="thigh_ixx" value="${(1.0/12.0) * thigh_mass * (3 * thigh_radius * thigh_radius + thigh_length * thigh_length)}" />

Commit message: Ajustar 4b: foot_height, foot_mass

File: robots/robot_stage4b.xacro (robot description, xacro)
@@ -56,7 +56,7 @@
   <xacro:property name="foot_length" value="0.35" />
   <xacro:property name="foot_width" value="0.15" />
-  <xacro:property name="foot_height" value="0.03" />
+  <xacro:property name="foot_height" value="0.05" />
   <xacro:property name="foot_offset_front" value="0.1" />
-  <xacro:property name="foot_mass" value="0.5" />
+  <xacro:property name="foot_mass" value="2.1" />
   <!-- Inertia for box (length, width, height): Ixx = (1/12)*m*(w^2+h^2); Iyy = (1/12)*m*(l^2+h^2); Izz = (1/12)*m*(l^2+w^2) -->
   <xacro:property name="foot_ixx" value="${(1.0/12.0) * foot_mass * (foot_width * foot_width + foot_height * foot_height)}" />
