Commit message: robo5 com braço fixo e ombro movel

File: robots/robot_stage5.xacro (robot description, xacro)
@@ -356,5 +356,5 @@
   <xacro:leg prefix="right" reflect="-1" />
   <xacro:leg prefix="left" reflect="1" />
-  <!-- Shoulder properties -->
+<!-- Shoulder properties -->
 <xacro:property name="shoulder_radius" value="0.04" />
 <xacro:property name="shoulder_length" value="0.1" />
@@ -370,5 +370,5 @@
 <xacro:property name="upper_arm_iyy" value="0.005" />
 <xacro:property name="upper_arm_izz" value="0.001" />
-<!-- Lower arm properties -->
+<!-- Lower arm properties (mantido para cálculo de massa, mas será fixo) -->
 <xacro:property name="lower_arm_radius" value="0.03" />
 <xacro:property name="lower_arm_length" value="0.22" />
@@ -377,5 +377,5 @@
 <xacro:property name="lower_arm_iyy" value="0.003" />
 <xacro:property name="lower_arm_izz" value="0.001" />
-<!-- Hand properties -->
+<!-- Hand properties (mantido para cálculo de massa, mas será fixo) -->
 <xacro:property name="hand_length" value="0.08" />
 <xacro:property name="hand_width" value="0.06" />
@@ -385,5 +385,5 @@
 <xacro:property name="hand_iyy" value="0.0001" />
 <xacro:property name="hand_izz" value="0.0001" />
-<!-- Arm macro -->
+<!-- Arm macro simplificado -->
 <xacro:macro name="arm" params="prefix reflect">
   <!-- Shoulder joint: base_link to shoulder (frontal movement) -->
@@ -393,5 +393,6 @@
     <origin xyz="0 ${(body_radius + shoulder_radius) * reflect} ${body_offset + body_length/4}" rpy="0 0 0"/>
     <axis xyz="0 1 0"/> <!-- Shoulder frontal movement -->
-    <limit lower="${-90 * deg_to_rad}" upper="${90 * deg_to_rad}" effort="100" velocity="3"/>
+    <!-- Limite de 45° para frente e trás -->
+    <limit lower="${-45 * deg_to_rad}" upper="${45 * deg_to_rad}" effort="100" velocity="3"/>
     <dynamics damping="${joint_dumping}" friction="${joint_friction}"/>
   </joint>
@@ -416,5 +417,5 @@
     </inertial>
   </link>
-  <!-- Shoulder joint: shoulder frontal to shoulder lateral -->
+  <!-- Shoulder joint: shoulder frontal to shoulder lateral (movimento lateral) -->
   <joint name="${prefix}_shoulder_front_to_lateral" type="revolute">
     <parent link="${prefix}_shoulder_front_link"/>
@@ -422,5 +423,6 @@
     <origin xyz="0 0 0" rpy="0 0 0"/>
     <axis xyz="1 0 0"/> <!-- Shoulder lateral movement -->
-    <limit lower="${-45 * deg_to_rad}" upper="${180 * deg_to_rad}" effort="80" velocity="3"/>
+    <!-- Limitar movimento lateral -->
+    <limit lower="${-10 * deg_to_rad}" upper="${45 * deg_to_rad}" effort="80" velocity="3"/>
     <dynamics damping="${joint_dumping}" friction="${joint_friction}"/>
   </joint>
@@ -445,17 +447,15 @@
     </inertial>
   </link>
-  <!-- Upper arm joint: shoulder to upper arm -->
-  <joint name="${prefix}_shoulder_to_upper_arm" type="revolute">
+  <!-- Upper arm joint: FIXO (sem movimento) -->
+  <joint name="${prefix}_shoulder_to_upper_arm" type="fixed">
     <parent link="${prefix}_shoulder_lateral_link"/>
     <child link="${prefix}_upper_arm_link"/>
+    <!-- Braço a 0° (para baixo) -->
     <origin xyz="0 0 0" rpy="0 0 0"/>
-    <axis xyz="0 1 0"/> <!-- Upper arm movement -->
-    <limit lower="${-120 * deg_to_rad}" upper="${30 * deg_to_rad}" effort="80" velocity="3"/>
-    <dynamics damping="${joint_dumping}" friction="${joint_friction}"/>
   </joint>
   <!-- Upper arm link -->
   <link name="${prefix}_upper_arm_link">
     <visual>
-      <origin rpy="0 ${90 * deg_to_rad} 0" xyz="0 0 ${-upper_arm_length/2}"/>
+      <origin rpy="0 0 0" xyz="0 0 ${-upper_arm_length/2}"/>
       <geometry>
         <cylinder length="${upper_arm_length}" radius="${upper_arm_radius}"/>
@@ -464,5 +464,5 @@
     </visual>
     <collision>
-      <origin rpy="0 ${90 * deg_to_rad} 0" xyz="0 0 ${-upper_arm_length/2}"/>
+      <origin rpy="0 0 0" xyz="0 0 ${-upper_arm_length/2}"/>
       <geometry>
         <cylinder length="${upper_arm_length}" radius="${upper_arm_radius}"/>
@@ -470,22 +470,20 @@
     </collision>
     <inertial>
-      <origin rpy="0 ${90 * deg_to_rad} 0" xyz="0 0 ${-upper_arm_length/2}"/>
+      <origin rpy="0 0 0" xyz="0 0 ${-upper_arm_length/2}"/>
       <mass value="${upper_arm_mass}"/>
       <inertia ixx="${upper_arm_ixx}" ixy="0.0" ixz="0.0" iyy="${upper_arm_iyy}" iyz="0.0" izz="${upper_arm_izz}"/>
     </inertial>
   </link>
-  <!-- Elbow joint: upper arm to lower arm -->
-  <joint name="${prefix}_upper_arm_to_lower_arm" type="revolute">
+  <!-- Elbow joint: FIXO (sem movimento) -->
+  <joint name="${prefix}_upper_arm_to_lower_arm" type="fixed">
     <parent link="${prefix}_upper_arm_link"/>
     <child link="${prefix}_lower_arm_link"/>
-    <origin xyz="0 0 ${-upper_arm_length}" rpy="0 0 0"/>
-    <axis xyz="0 1 0"/> <!-- Elbow flexion/extension -->
-    <limit lower="${0 * deg_to_rad}" upper="${150 * deg_to_rad}" effort="60" velocity="3"/>
-    <dynamics damping="${joint_dumping}" friction="${joint_friction}"/>
+    <!-- Antebraço a 90° (para frente) -->
+    <origin xyz="0 0 ${-upper_arm_length}" rpy="0 ${-90 * deg_to_rad} 0"/>
   </joint>
   <!-- Lower arm link -->
   <link name="${prefix}_lower_arm_link">
     <visual>
-      <origin rpy="0 ${90 * deg_to_rad} 0" xyz="0 0 ${-lower_arm_length/2}"/>
+      <origin rpy="0 0 0" xyz="0 0 ${-lower_arm_length/2}"/>
       <geometry>
         <cylinder length="${lower_arm_length}" radius="${lower_arm_radius}"/>
@@ -494,5 +492,5 @@
     </visual>
     <collision>
-      <origin rpy="0 ${90 * deg_to_rad} 0" xyz="0 0 ${-lower_arm_length/2}"/>
+      <origin rpy="0 0 0" xyz="0 0 ${-lower_arm_length/2}"/>
       <geometry>
         <cylinder length="${lower_arm_length}" radius="${lower_arm_radius}"/>
@@ -500,17 +498,14 @@
     </collision>
     <inertial>
-      <origin rpy="0 ${90 * deg_to_rad} 0" xyz="0 0 ${-lower_arm_length/2}"/>
+      <origin rpy="0 0 0" xyz="0 0 ${-lower_arm_length/2}"/>
       <mass value="${lower_arm_mass}"/>
       <inertia ixx="${lower_arm_ixx}" ixy="0.0" ixz="0.0" iyy="${lower_arm_iyy}" iyz="0.0" izz="${lower_arm_izz}"/>
     </inertial>
   </link>
-  <!-- Wrist joint: lower arm to hand -->
-  <joint name="${prefix}_lower_arm_to_hand" type="revolute">
+  <!-- Wrist joint: FIXO (sem movimento) -->
+  <joint name="${prefix}_lower_arm_to_hand" type="fixed">
     <parent link="${prefix}_lower_arm_link"/>
     <child link="${prefix}_hand_link"/>
     <origin xyz="0 0 ${-lower_arm_length}" rpy="0 0 0"/>
-    <axis xyz="0 1 0"/> <!-- Wrist movement -->
-    <limit lower="${-30 * deg_to_rad}" upper="${30 * deg_to_rad}" effort="40" velocity="3"/>
-    <dynamics damping="${joint_dumping}" friction="${joint_friction}"/>
   </joint>
   <!-- Hand link -->

Commit message: alterado medidas do robo5

File: robots/robot_stage5.xacro (robot description, xacro)
@@ -2,6 +2,6 @@
 <robot xmlns:xacro="http://www.ros.org/wiki/xacro" name="myrobot_st4">
   <!-- Body properties -->
-  <xacro:property name="body_radius" value="0.15" />
-  <xacro:property name="body_length" value="0.3" />
+  <xacro:property name="body_radius" value="0.12" />
+  <xacro:property name="body_length" value="0.4" />
   <xacro:property name="body_mass" value="5.0" />
   <xacro:property name="body_ixx" value="0.1" />
@@ -50,9 +50,38 @@
   <xacro:property name="foot_izz" value="0.0005" />
   <!-- Head properties -->
-  <xacro:property name="head_radius" value="0.1" />
-  <xacro:property name="head_mass" value="1.0" />
+  <xacro:property name="head_radius" value="0.08" />
+  <xacro:property name="head_mass" value="0.8" />
   <xacro:property name="head_ixx" value="0.005" />
   <xacro:property name="head_iyy" value="0.005" />
   <xacro:property name="head_izz" value="0.005" />
+  <!-- Shoulder properties -->
+<xacro:property name="shoulder_radius" value="0.03" />
+<xacro:property name="shoulder_length" value="0.06" />
+<xacro:property name="shoulder_mass" value="0.2" />
+<xacro:property name="shoulder_ixx" value="0.001" />
+<xacro:property name="shoulder_iyy" value="0.001" />
+<xacro:property name="shoulder_izz" value="0.001" />
+<!-- Upper arm properties -->
+<xacro:property name="upper_arm_radius" value="0.025" />
+<xacro:property name="upper_arm_length" value="0.18" />
+<xacro:property name="upper_arm_mass" value="0.5" />
+<xacro:property name="upper_arm_ixx" value="0.005" />
+<xacro:property name="upper_arm_iyy" value="0.005" />
+<xacro:property name="upper_arm_izz" value="0.001" />
+<!-- Lower arm properties (mantido para cálculo de massa, mas será fixo) -->
+<xacro:property name="lower_arm_radius" value="0.02" />
+<xacro:property name="lower_arm_length" value="0.16" />
+<xacro:property name="lower_arm_mass" value="0.4" />
+<xacro:property name="lower_arm_ixx" value="0.003" />
+<xacro:property name="lower_arm_iyy" value="0.003" />
+<xacro:property name="lower_arm_izz" value="0.001" />
+<!-- Hand properties (mantido para cálculo de massa, mas será fixo) -->
+<xacro:property name="hand_length" value="0.06" />
+<xacro:property name="hand_width" value="0.04" />
+<xacro:property name="hand_height" value="0.03" />
+<xacro:property name="hand_mass" value="0.1" />
+<xacro:property name="hand_ixx" value="0.0001" />
+<xacro:property name="hand_iyy" value="0.0001" />
+<xacro:property name="hand_izz" value="0.0001" />
   <!-- IMU properties -->
   <xacro:property name="imu_length" value="0.02" />
@@ -157,5 +186,5 @@
     <!-- Z: Como o corpo principal e posicionado em 0 0 0, body_offset move a joint para o centro do corpo -->
     <!-- Z: body_length/2 move a joint para o topo do corpo -->
-	  <origin xyz="0 0 ${body_offset + body_length/2}"/>
+	  <origin xyz="0 0 ${body_offset + body_length/2 + head_radius}"/>
   </joint>
   <!-- Leg macro (creates left/right leg: thigh, shin, foot) -->
@@ -356,33 +385,4 @@
   <xacro:leg prefix="right" reflect="-1" />
   <xacro:leg prefix="left" reflect="1" />
-<!-- Shoulder properties -->
-<xacro:property name="shoulder_radius" value="0.04" />
-<xacro:property name="shoulder_length" value="0.1" />
-<xacro:property name="shoulder_mass" value="0.3" />
-<xacro:property name="shoulder_ixx" value="0.001" />
-<xacro:property name="shoulder_iyy" value="0.001" />
-<xacro:property name="shoulder_izz" value="0.001" />
-<!-- Upper arm properties -->
-<xacro:property name="upper_arm_radius" value="0.035" />
-<xacro:property name="upper_arm_length" value="0.25" />
-<xacro:property name="upper_arm_mass" value="0.8" />
-<xacro:property name="upper_arm_ixx" value="0.005" />
-<xacro:property name="upper_arm_iyy" value="0.005" />
-<xacro:property name="upper_arm_izz" value="0.001" />
-<!-- Lower arm properties (mantido para cálculo de massa, mas será fixo) -->
-<xacro:property name="lower_arm_radius" value="0.03" />
-<xacro:property name="lower_arm_length" value="0.22" />
-<xacro:property name="lower_arm_mass" value="0.6" />
-<xacro:property name="lower_arm_ixx" value="0.003" />
-<xacro:property name="lower_arm_iyy" value="0.003" />
-<xacro:property name="lower_arm_izz" value="0.001" />
-<!-- Hand properties (mantido para cálculo de massa, mas será fixo) -->
-<xacro:property name="hand_length" value="0.08" />
-<xacro:property name="hand_width" value="0.06" />
-<xacro:property name="hand_height" value="0.04" />
-<xacro:property name="hand_mass" value="0.2" />
-<xacro:property name="hand_ixx" value="0.0001" />
-<xacro:property name="hand_iyy" value="0.0001" />
-<xacro:property name="hand_izz" value="0.0001" />
 <!-- Arm macro simplificado -->
 <xacro:macro name="arm" params="prefix reflect">
@@ -391,5 +391,5 @@
     <parent link="base_link"/>
     <child link="${prefix}_shoulder_front_link"/>
-    <origin xyz="0 ${(body_radius + shoulder_radius) * reflect} ${body_offset + body_length/4}" rpy="0 0 0"/>
+    <origin xyz="0 ${(body_radius + shoulder_radius) * reflect} ${body_offset + body_length/2 - shoulder_radius}" rpy="0 0 0"/>
     <axis xyz="0 1 0"/> <!-- Shoulder frontal movement -->
     <!-- Limite de 45° para frente e trás -->

Commit message: corrigi bugs

File: robots/robot_stage5.xacro (robot description, xacro)
@@ -1,4 +1,15 @@
 <?xml version="1.0"?>
 <robot xmlns:xacro="http://www.ros.org/wiki/xacro" name="myrobot_st4">
+<!-- ORIENTACAO INICIAL  -->
+<xacro:property name="initial_roll" value="0.0" />
+<xacro:property name="initial_pitch" value="0.14" />
+<xacro:property name="initial_yaw" value="0.0" />
+<!-- CONFIGURACOES INICIAIS PARA EQUILIBRIO E CAMINHADA -->
+<xacro:property name="initial_hip_frontal" value="0.0" />
+<xacro:property name="initial_hip_lateral" value="0.0" />
+<xacro:property name="initial_knee" value="0.5" />
+<xacro:property name="initial_ankle_frontal" value="-0.25" />
+<xacro:property name="initial_ankle_lateral" value="0.0" />
+<xacro:property name="initial_pitch" value="0.15" />
   <!-- Body properties -->
   <xacro:property name="body_radius" value="0.12" />
@@ -69,5 +80,5 @@
 <xacro:property name="upper_arm_iyy" value="0.005" />
 <xacro:property name="upper_arm_izz" value="0.001" />
-<!-- Lower arm properties (mantido para cálculo de massa, mas será fixo) -->
+<!-- Lower arm properties (mantido para calculo de massa, mas sera fixo) -->
 <xacro:property name="lower_arm_radius" value="0.02" />
 <xacro:property name="lower_arm_length" value="0.16" />
@@ -76,5 +87,5 @@
 <xacro:property name="lower_arm_iyy" value="0.003" />
 <xacro:property name="lower_arm_izz" value="0.001" />
-<!-- Hand properties (mantido para cálculo de massa, mas será fixo) -->
+<!-- Hand properties (mantido para calculo de massa, mas sera fixo) -->
 <xacro:property name="hand_length" value="0.06" />
 <xacro:property name="hand_width" value="0.04" />
@@ -191,15 +202,11 @@
     <!-- Hip joint: base_link to hip ball -->
     <joint name="base_to_${prefix}_hip_ball" type="revolute">
-      <parent link="base_link"/>
-      <child link="${prefix}_hip_ball_link"/>
-      <!-- Z: Como o corpo principal e posicionado em 0 0 0, body_offset move o centro da esfera/articulacao para o centro do corpo -->
-      <!-- Z: Diminuir body_length/2 move o centro da esfera/articulacao para a base inferior do corpo -->
-      <!-- Y: body_radius posiciona o centro da esfera/articulacao do quadril na borda do corpo -->
-      <!-- Y: hip_radius tira a esfera/articulacao de dentro do corpo, caso contrario metade da esfera/articulacao ficaria dentro do corpo -->
-      <origin xyz="0 ${(body_radius + hip_radius) * reflect} ${body_offset - body_length/2}"/>
-      <axis xyz="0 1 0"/> <!-- Movimento frontal -->
-      <limit lower="${-75 * deg_to_rad}" upper="${60 * deg_to_rad}" effort="1000" velocity="5"/>
-      <dynamics damping="${joint_damping}" friction="${joint_friction}"/>
-    </joint>
+  <parent link="base_link"/>
+  <child link="${prefix}_hip_ball_link"/>
+  <origin xyz="0 ${(body_radius + hip_radius) * reflect} ${body_offset - body_length/2}"/>
+  <axis xyz="0 1 0"/>
+  <limit lower="${-75 * deg_to_rad}" upper="${60 * deg_to_rad}" effort="1000" velocity="5"/>
+  <dynamics damping="${joint_damping}" friction="${joint_friction}"/>
+</joint>
     <!-- Hip Ball -->
     <link name="${prefix}_hip_ball_link">
@@ -285,11 +292,11 @@
     <!-- Knee joint: knee ball to shin -->
     <joint name="${prefix}_knee_ball_to_shin" type="revolute">
-      <parent link="${prefix}_knee_ball_link"/>
-      <child link="${prefix}_shin_link"/>
-      <origin xyz="0 0 0"/>
-      <axis xyz="0 1 0"/>
-      <limit lower="${0 * deg_to_rad}" upper="${90 * deg_to_rad}" effort="1000" velocity="5"/>
-      <dynamics damping="${joint_damping}" friction="${joint_friction}"/>
-    </joint>
+  <parent link="${prefix}_knee_ball_link"/>
+  <child link="${prefix}_shin_link"/>
+  <origin xyz="0 0 0"/>
+  <axis xyz="0 1 0"/>
+  <limit lower="${0 * deg_to_rad}" upper="${90 * deg_to_rad}" effort="1000" velocity="5"/>
+  <dynamics damping="${joint_damping}" friction="${joint_friction}"/>
+</joint>
     <!-- Shin -->
     <link name="${prefix}_shin_link">
@@ -317,14 +324,11 @@
     <!-- Ankle joint: shin to ankle ball -->
     <joint name="${prefix}_shin_to_ankle_ball" type="revolute">
-      <parent link="${prefix}_shin_link"/>
-      <child link="${prefix}_ankle_ball_link"/>
-      <!-- Z: Como o parent e a canela, o centro da esfera/articulacao do tornozelo coincide inicialmente com sua referencia que é o knee joint -->
-      <!-- Z: Diminuir knee_radius + shin_length faz o centro da esfera/articulacao do tornozelo coincidir com a base inferior da canela -->
-      <!-- Z: Diminuir ankle_radius faz o topo da esfera/articulacao do tornozelo coincidir com a base inferior da canela -->
-      <origin xyz="0 0 ${-knee_radius - shin_length - ankle_radius}"/>
-      <axis xyz="0 1 0"/> <!-- Movimento frontal -->
-      <limit lower="${-30 * deg_to_rad}" upper="${75 * deg_to_rad}" effort="1000" velocity="5"/>
-      <dynamics damping="${joint_damping}" friction="${joint_friction}"/>
-    </joint>
+  <parent link="${prefix}_shin_link"/>
+  <child link="${prefix}_ankle_ball_link"/>
+  <origin xyz="0 0 ${-knee_radius - shin_length - ankle_radius}"/>
+  <axis xyz="0 1 0"/>
+  <limit lower="${-30 * deg_to_rad}" upper="${75 * deg_to_rad}" effort="1000" velocity="5"/>
+  <dynamics damping="${joint_damping}" friction="${joint_friction}"/>
+</joint>
     <!-- Ankle Ball -->
     <link name="${prefix}_ankle_ball_link">
@@ -530,4 +534,12 @@
   </link>
 </xacro:macro>
+ <!-- Configurações iniciais das juntas para maior estabilidade -->
+<xacro:property name="initial_hip_frontal" value="0.0" />
+<xacro:property name="initial_hip_lateral" value="0.0" />
+<xacro:property name="initial_knee" value="0.4" />
+<xacro:property name="initial_ankle_frontal" value="-0.15" />
+<xacro:property name="initial_ankle_lateral" value="0.0" />
+<!-- Pequena inclinação frontal adicional do corpo -->
+<xacro:property name="initial_pitch" value="0.1" />
 <!-- Instantiate arms -->
 <xacro:arm prefix="right" reflect="-1"/>
