Commit message: Remover massa de articulações do robô 5

File: robots/robot_stage5.xacro (robot description, xacro)
@@ -24,5 +24,5 @@
   <!-- Hip properties -->
   <xacro:property name="hip_radius" value="0.05" />
-  <xacro:property name="hip_mass" value="0.5" />
+  <xacro:property name="hip_mass" value="0.0" />
   <xacro:property name="hip_ixx" value="${0.4 * hip_mass * hip_radius * hip_radius}" />
   <xacro:property name="hip_iyy" value="${0.4 * hip_mass * hip_radius * hip_radius}" />
@@ -37,5 +37,5 @@
   <!-- Knee properties -->
   <xacro:property name="knee_radius" value="0.04" />
-  <xacro:property name="knee_mass" value="0.5" />
+  <xacro:property name="knee_mass" value="0.0" />
   <xacro:property name="knee_ixx" value="${0.4 * knee_mass * knee_radius * knee_radius}" />
   <xacro:property name="knee_iyy" value="${0.4 * knee_mass * knee_radius * knee_radius}" />
@@ -50,5 +50,5 @@
   <!-- Ankle properties -->
   <xacro:property name="ankle_radius" value="0.03" />
-  <xacro:property name="ankle_mass" value="0.5" />
+  <xacro:property name="ankle_mass" value="0.0" />
   <xacro:property name="ankle_ixx" value="${0.4 * ankle_mass * ankle_radius * ankle_radius}" />
   <xacro:property name="ankle_iyy" value="${0.4 * ankle_mass * ankle_radius * ankle_radius}" />
@@ -65,5 +65,5 @@
   <!-- Shoulder properties -->
   <xacro:property name="shoulder_radius" value="0.04" />
-  <xacro:property name="shoulder_mass" value="0.5" />
+  <xacro:property name="shoulder_mass" value="0.0" />
   <xacro:property name="shoulder_ixx" value="${0.4 * shoulder_mass * shoulder_radius * shoulder_radius}" />
   <xacro:property name="shoulder_iyy" value="${0.4 * shoulder_mass * shoulder_radius * shoulder_radius}" />

Commit message: Arrumar altura do robô 5

File: robots/robot_stage5.xacro (robot description, xacro)
@@ -113,5 +113,5 @@
   </material>
   <!-- Altura total -->
-  <xacro:property name="leg_total_length" value="${hip_radius + thigh_length + 2 * knee_radius + shin_length + 2 * ankle_radius + foot_height}" />
+  <xacro:property name="leg_total_length" value="${thigh_length + shin_length + foot_height}" />
   <xacro:property name="body_offset" value="${body_length/2 + leg_total_length}" />
   <xacro:property name="deg_to_rad" value="${3.14159 / 180}" />

Commit message: ajuste no robo

File: robots/robot_stage5.xacro (robot description, xacro)
@@ -4,5 +4,5 @@
   <xacro:property name="body_radius" value="0.15" />
   <xacro:property name="body_length" value="0.50" />
-  <xacro:property name="body_mass" value="35.1" />
+  <xacro:property name="body_mass" value="35.7" />
   <!-- Inertia for solid cylinder (axis z): Ixx = Iyy = (1/12)*m*(3*r^2+h^2); Izz = (1/2)*m*r^2 -->
   <xacro:property name="body_ixx" value="${(1.0/12.0) * body_mass * (3 * body_radius * body_radius + body_length * body_length)}" />
@@ -24,5 +24,5 @@
   <!-- Hip properties -->
   <xacro:property name="hip_radius" value="0.05" />
-  <xacro:property name="hip_mass" value="0.0" />
+  <xacro:property name="hip_mass" value="0.8" />
   <xacro:property name="hip_ixx" value="${0.4 * hip_mass * hip_radius * hip_radius}" />
   <xacro:property name="hip_iyy" value="${0.4 * hip_mass * hip_radius * hip_radius}" />
@@ -31,5 +31,5 @@
   <xacro:property name="thigh_radius" value="0.075" />
   <xacro:property name="thigh_length" value="0.40" />
-  <xacro:property name="thigh_mass" value="18.5" />
+  <xacro:property name="thigh_mass" value="19.0" />
   <xacro:property name="thigh_ixx" value="${(1.0/12.0) * thigh_mass * (3 * thigh_radius * thigh_radius + thigh_length * thigh_length)}" />
   <xacro:property name="thigh_iyy" value="${(1.0/12.0) * thigh_mass * (3 * thigh_radius * thigh_radius + thigh_length * thigh_length)}" />
@@ -37,5 +37,5 @@
   <!-- Knee properties -->
   <xacro:property name="knee_radius" value="0.04" />
-  <xacro:property name="knee_mass" value="0.0" />
+  <xacro:property name="knee_mass" value="0.4" />
   <xacro:property name="knee_ixx" value="${0.4 * knee_mass * knee_radius * knee_radius}" />
   <xacro:property name="knee_iyy" value="${0.4 * knee_mass * knee_radius * knee_radius}" />
@@ -44,5 +44,5 @@
   <xacro:property name="shin_radius" value="0.06" />
   <xacro:property name="shin_length" value="0.43" />
-  <xacro:property name="shin_mass" value="7.6" />
+  <xacro:property name="shin_mass" value="8.09" />
   <xacro:property name="shin_ixx" value="${(1.0/12.0) * shin_mass * (3 * shin_radius * shin_radius + shin_length * shin_length)}" />
   <xacro:property name="shin_iyy" value="${(1.0/12.0) * shin_mass * (3 * shin_radius * shin_radius + shin_length * shin_length)}" />
@@ -50,5 +50,5 @@
   <!-- Ankle properties -->
   <xacro:property name="ankle_radius" value="0.03" />
-  <xacro:property name="ankle_mass" value="0.0" />
+  <xacro:property name="ankle_mass" value="0.3" />
   <xacro:property name="ankle_ixx" value="${0.4 * ankle_mass * ankle_radius * ankle_radius}" />
   <xacro:property name="ankle_iyy" value="${0.4 * ankle_mass * ankle_radius * ankle_radius}" />
@@ -65,5 +65,5 @@
   <!-- Shoulder properties -->
   <xacro:property name="shoulder_radius" value="0.04" />
-  <xacro:property name="shoulder_mass" value="0.0" />
+  <xacro:property name="shoulder_mass" value="0.5" />
   <xacro:property name="shoulder_ixx" value="${0.4 * shoulder_mass * shoulder_radius * shoulder_radius}" />
   <xacro:property name="shoulder_iyy" value="${0.4 * shoulder_mass * shoulder_radius * shoulder_radius}" />
@@ -530,5 +530,5 @@
     <link name="${prefix}_hand_link">
       <visual>
-        <origin rpy="0 0 0" xyz="0 0 ${-hand_height/2}"/>
+        <origin rpy="${90 * deg_to_rad} 0 0" xyz="${hand_length/2} 0 0"/>
         <geometry>
           <box size="${hand_length} ${hand_width} ${hand_height}"/>
@@ -537,5 +537,5 @@
       </visual>
       <collision>
-        <origin rpy="0 0 0" xyz="0 0 ${-hand_height/2}"/>
+        <origin rpy="${90 * deg_to_rad} 0 0" xyz="${hand_length/2} 0 0"/>
         <geometry>
           <box size="${hand_length} ${hand_width} ${hand_height}"/>
@@ -543,5 +543,5 @@
       </collision>
       <inertial>
-        <origin rpy="0 0 0" xyz="0 0 ${-hand_height/2}"/>
+        <origin rpy="${90 * deg_to_rad} 0 0" xyz="${hand_length/2} 0 0"/>
         <mass value="${hand_mass}"/>
         <inertia ixx="${hand_ixx}" ixy="0.0" ixz="0.0" iyy="${hand_iyy}" iyz="0.0" izz="${hand_izz}"/>

Commit message: Arrumar mão

File: robots/robot_stage5.xacro (robot description, xacro)
@@ -530,18 +530,18 @@
     <link name="${prefix}_hand_link">
       <visual>
-        <origin rpy="${90 * deg_to_rad} 0 0" xyz="${hand_length/2} 0 0"/>
-        <geometry>
-          <box size="${hand_length} ${hand_width} ${hand_height}"/>
-        </geometry>
-        <material name="robot_material_2"/>
-      </visual>
-      <collision>
-        <origin rpy="${90 * deg_to_rad} 0 0" xyz="${hand_length/2} 0 0"/>
-        <geometry>
-          <box size="${hand_length} ${hand_width} ${hand_height}"/>
-        </geometry>
-      </collision>
-      <inertial>
-        <origin rpy="${90 * deg_to_rad} 0 0" xyz="${hand_length/2} 0 0"/>
+        <origin rpy="0 0 0" xyz="0 0 ${-hand_length/4}"/>
+        <geometry>
+          <box size="${hand_width} ${hand_height} ${hand_length}"/>
+        </geometry>
+        <material name="robot_material_2"/>
+      </visual>
+      <collision>
+        <origin rpy="0 0 0" xyz="0 0 ${-hand_length/4}"/>
+        <geometry>
+          <box size="${hand_width} ${hand_height} ${hand_length}"/>
+        </geometry>
+      </collision>
+      <inertial>
+        <origin rpy="0 0 0" xyz="0 0 ${-hand_length/4}"/>
         <mass value="${hand_mass}"/>
         <inertia ixx="${hand_ixx}" ixy="0.0" ixz="0.0" iyy="${hand_iyy}" iyz="0.0" izz="${hand_izz}"/>

Commit message: to treinando cc,pba,pg

File: robots/robot_stage5.xacro (robot description, xacro)
@@ -4,5 +4,5 @@
   <xacro:property name="body_radius" value="0.15" />
   <xacro:property name="body_length" value="0.50" />
-  <xacro:property name="body_mass" value="35.7" />
+  <xacro:property name="body_mass" value="37.69" />
   <!-- Inertia for solid cylinder (axis z): Ixx = Iyy = (1/12)*m*(3*r^2+h^2); Izz = (1/2)*m*r^2 -->
   <xacro:property name="body_ixx" value="${(1.0/12.0) * body_mass * (3 * body_radius * body_radius + body_length * body_length)}" />
@@ -31,5 +31,5 @@
   <xacro:property name="thigh_radius" value="0.075" />
   <xacro:property name="thigh_length" value="0.40" />
-  <xacro:property name="thigh_mass" value="19.0" />
+  <xacro:property name="thigh_mass" value="18.0" />
   <xacro:property name="thigh_ixx" value="${(1.0/12.0) * thigh_mass * (3 * thigh_radius * thigh_radius + thigh_length * thigh_length)}" />
   <xacro:property name="thigh_iyy" value="${(1.0/12.0) * thigh_mass * (3 * thigh_radius * thigh_radius + thigh_length * thigh_length)}" />
@@ -44,5 +44,5 @@
   <xacro:property name="shin_radius" value="0.06" />
   <xacro:property name="shin_length" value="0.43" />
-  <xacro:property name="shin_mass" value="8.09" />
+  <xacro:property name="shin_mass" value="8.1" />
   <xacro:property name="shin_ixx" value="${(1.0/12.0) * shin_mass * (3 * shin_radius * shin_radius + shin_length * shin_length)}" />
   <xacro:property name="shin_iyy" value="${(1.0/12.0) * shin_mass * (3 * shin_radius * shin_radius + shin_length * shin_length)}" />

Commit message: Ajustar aparência do robô

File: robots/robot_stage5.xacro (robot description, xacro)
@@ -105,10 +105,23 @@
   <xacro:property name="joint_velocity" value="3.0" />
   <xacro:property name="position_gain" value="0.5" />
-  <!-- Materials -->
-  <material name="robot_material_1">
-    <color rgba="0.7 0.7 0.8 1"/>
+  <!-- Estrutura principal (tronco, base) -->
+  <material name="mat_structure">
+      <color rgba="0.35 0.35 0.37 1.0"/>
   </material>
-  <material name="robot_material_2">
-    <color rgba="0.9 0.9 1.0 1"/>
+  <!-- Membros (pernas, braços, cabeça...) -->
+  <material name="mat_limb">
+      <color rgba="0.70 0.70 0.72 1.0"/>
+  </material>
+  <!-- Articulacoes (esferas, joints visuais) -->
+  <material name="mat_joint">
+      <color rgba="0.45 0.45 0.47 1.0"/>
+  </material>
+  <!-- Sensor IMU -->
+  <material name="mat_sensor">
+      <color rgba="0.25 0.55 0.45 1.0"/>
+  </material>
+  <!-- Pes / contato com o solo -->
+  <material name="mat_foot">
+      <color rgba="0.10 0.10 0.10 1.0"/>
   </material>
   <!-- Altura total -->
@@ -123,5 +136,5 @@
         <cylinder length="${body_length}" radius="${body_radius}"/>
       </geometry>
-      <material name="robot_material_1"/>
+      <material name="mat_structure"/>
     </visual>
     <collision>
@@ -144,5 +157,5 @@
         <box size="${imu_length} ${imu_width} ${imu_height}"/>
       </geometry>
-      <material name="robot_material_2"/>
+      <material name="mat_sensor"/>
     </visual>
     <collision>
@@ -169,5 +182,5 @@
         <cylinder length="${neck_length}" radius="${neck_radius}"/>
       </geometry>
-      <material name="robot_material_2"/>
+      <material name="mat_limb"/>
     </visual>
     <collision>
@@ -196,5 +209,5 @@
         <sphere radius="${head_radius}"/>
       </geometry>
-      <material name="robot_material_2"/>
+      <material name="mat_limb"/>
     </visual>
     <collision>
@@ -234,5 +247,5 @@
           <sphere radius="${hip_radius}"/>
         </geometry>
-        <material name="robot_material_2"/>
+        <material name="mat_joint"/>
       </visual>
       <collision>
@@ -262,5 +275,5 @@
           <sphere radius="${hip_radius * 0.5}"/>
         </geometry>
-        <material name="robot_material_2"/>
+        <material name="mat_joint"/>
       </visual>
       <inertial>
@@ -284,5 +297,5 @@
           <sphere radius="${hip_radius * 0.3}"/>
         </geometry>
-        <material name="robot_material_2"/>
+        <material name="mat_joint"/>
       </visual>
       <inertial>
@@ -304,5 +317,5 @@
           <cylinder length="${thigh_length}" radius="${thigh_radius}"/>
         </geometry>
-        <material name="robot_material_2"/>
+        <material name="mat_limb"/>
       </visual>
       <collision>
@@ -331,5 +344,5 @@
           <sphere radius="${knee_radius}"/>
         </geometry>
-        <material name="robot_material_2"/>
+        <material name="mat_joint"/>
       </visual>
       <collision>
@@ -360,5 +373,5 @@
           <cylinder length="${shin_length}" radius="${shin_radius}"/>
         </geometry>
-        <material name="robot_material_1"/>
+        <material name="mat_limb"/>
       </visual>
       <collision>
@@ -390,5 +403,5 @@
           <sphere radius="${ankle_radius}"/>
         </geometry>
-        <material name="robot_material_2"/>
+        <material name="mat_joint"/>
       </visual>
       <collision>
@@ -419,5 +432,5 @@
           <box size="${foot_length} ${foot_width} ${foot_height}"/>
         </geometry>
-        <material name="robot_material_2"/>
+        <material name="mat_foot"/>
       </visual>
       <collision>
@@ -453,5 +466,5 @@
           <sphere radius="${shoulder_radius}"/>
         </geometry>
-        <material name="robot_material_2"/>
+        <material name="mat_joint"/>
       </visual>
       <collision>
@@ -479,5 +492,5 @@
           <cylinder length="${arm_length}" radius="${arm_radius}"/>
         </geometry>
-        <material name="robot_material_2"/>
+        <material name="mat_limb"/>
       </visual>
       <collision>
@@ -507,5 +520,5 @@
           <cylinder length="${forearm_length}" radius="${forearm_radius}"/>
         </geometry>
-        <material name="robot_material_1"/>
+        <material name="mat_limb"/>
       </visual>
       <collision>
@@ -534,5 +547,5 @@
           <box size="${hand_width} ${hand_height} ${hand_length}"/>
         </geometry>
-        <material name="robot_material_2"/>
+        <material name="mat_limb"/>
       </visual>
       <collision>

Commit message: tentar fazer subir a rampa

File: robots/robot_stage5.xacro (robot description, xacro)
@@ -393,5 +393,5 @@
       <origin xyz="0 0 ${-shin_length}"/>
       <axis xyz="0 1 0"/>
-      <limit lower="${-20 * deg_to_rad}" upper="${20 * deg_to_rad}" effort="${joint_effort}" velocity="${joint_velocity}"/>
+      <limit lower="${-25 * deg_to_rad}" upper="${25 * deg_to_rad}" effort="${joint_effort}" velocity="${joint_velocity}"/>
       <dynamics damping="${joint_damping}" friction="${joint_friction}"/>
     </joint>
@@ -422,5 +422,5 @@
       <origin xyz="0 0 0"/>
       <axis xyz="1 0 0"/>
-      <limit lower="${-10 * deg_to_rad}" upper="${10 * deg_to_rad}" effort="${joint_effort}" velocity="${joint_velocity}"/>
+      <limit lower="${-15 * deg_to_rad}" upper="${15 * deg_to_rad}" effort="${joint_effort}" velocity="${joint_velocity}"/>
       <dynamics damping="${joint_damping}" friction="${joint_friction}"/>
     </joint>

Commit message: ajuste da reunião

File: robots/robot_stage5.xacro (robot description, xacro)
@@ -55,6 +55,6 @@
   <xacro:property name="ankle_izz" value="${0.4 * ankle_mass * ankle_radius * ankle_radius}" />
   <!-- Foot properties -->
-  <xacro:property name="foot_length" value="0.25" />
-  <xacro:property name="foot_width" value="0.10" />
+  <xacro:property name="foot_length" value="0.30" />
+  <xacro:property name="foot_width" value="0.11" />
   <xacro:property name="foot_height" value="0.05" />
   <xacro:property name="foot_offset_front" value="0.05" />

Commit message: Update robot_stage5.xacro

File: robots/robot_stage5.xacro (robot description, xacro)
@@ -4,5 +4,5 @@
   <xacro:property name="body_radius" value="0.15" />
   <xacro:property name="body_length" value="0.50" />
-  <xacro:property name="body_mass" value="37.69" />
+  <xacro:property name="body_mass" value="34.49" />
   <!-- Inertia for solid cylinder (axis z): Ixx = Iyy = (1/12)*m*(3*r^2+h^2); Izz = (1/2)*m*r^2 -->
   <xacro:property name="body_ixx" value="${(1.0/12.0) * body_mass * (3 * body_radius * body_radius + body_length * body_length)}" />
@@ -12,5 +12,5 @@
   <xacro:property name="neck_radius" value="0.06" />
   <xacro:property name="neck_length" value="0.10" />
-  <xacro:property name="neck_mass" value="1.0" />
+  <xacro:property name="neck_mass" value="0.9" />
   <xacro:property name="neck_ixx" value="${(1.0/12.0) * neck_mass * (3 * neck_radius * neck_radius + neck_length * neck_length)}" />
   <xacro:property name="neck_iyy" value="${(1.0/12.0) * neck_mass * (3 * neck_radius * neck_radius + neck_length * neck_length)}" />
@@ -18,5 +18,5 @@
   <!-- Head properties -->
   <xacro:property name="head_radius" value="0.09" />
-  <xacro:property name="head_mass" value="4.5" />
+  <xacro:property name="head_mass" value="4.1" />
   <xacro:property name="head_ixx" value="${0.4 * head_mass * head_radius * head_radius}" />
   <xacro:property name="head_iyy" value="${0.4 * head_mass * head_radius * head_radius}" />
@@ -24,5 +24,5 @@
   <!-- Hip properties -->
   <xacro:property name="hip_radius" value="0.05" />
-  <xacro:property name="hip_mass" value="0.8" />
+  <xacro:property name="hip_mass" value="0.7" />
   <xacro:property name="hip_ixx" value="${0.4 * hip_mass * hip_radius * hip_radius}" />
   <xacro:property name="hip_iyy" value="${0.4 * hip_mass * hip_radius * hip_radius}" />
@@ -31,5 +31,5 @@
   <xacro:property name="thigh_radius" value="0.075" />
   <xacro:property name="thigh_length" value="0.40" />
-  <xacro:property name="thigh_mass" value="18.0" />
+  <xacro:property name="thigh_mass" value="16.0" />
   <xacro:property name="thigh_ixx" value="${(1.0/12.0) * thigh_mass * (3 * thigh_radius * thigh_radius + thigh_length * thigh_length)}" />
   <xacro:property name="thigh_iyy" value="${(1.0/12.0) * thigh_mass * (3 * thigh_radius * thigh_radius + thigh_length * thigh_length)}" />
@@ -37,5 +37,5 @@
   <!-- Knee properties -->
   <xacro:property name="knee_radius" value="0.04" />
-  <xacro:property name="knee_mass" value="0.4" />
+  <xacro:property name="knee_mass" value="0.35" />
   <xacro:property name="knee_ixx" value="${0.4 * knee_mass * knee_radius * knee_radius}" />
   <xacro:property name="knee_iyy" value="${0.4 * knee_mass * knee_radius * knee_radius}" />
@@ -44,5 +44,5 @@
   <xacro:property name="shin_radius" value="0.06" />
   <xacro:property name="shin_length" value="0.43" />
-  <xacro:property name="shin_mass" value="8.1" />
+  <xacro:property name="shin_mass" value="7.3" />
   <xacro:property name="shin_ixx" value="${(1.0/12.0) * shin_mass * (3 * shin_radius * shin_radius + shin_length * shin_length)}" />
   <xacro:property name="shin_iyy" value="${(1.0/12.0) * shin_mass * (3 * shin_radius * shin_radius + shin_length * shin_length)}" />
@@ -59,5 +59,5 @@
   <xacro:property name="foot_height" value="0.05" />
   <xacro:property name="foot_offset_front" value="0.05" />
-  <xacro:property name="foot_mass" value="2.1" />
+  <xacro:property name="foot_mass" value="2.0" />
   <xacro:property name="foot_ixx" value="${(1.0/12.0) * foot_mass * (foot_width * foot_width + foot_height * foot_height)}" />
   <xacro:property name="foot_iyy" value="${(1.0/12.0) * foot_mass * (foot_length * foot_length + foot_height * foot_height)}" />
@@ -72,5 +72,5 @@
   <xacro:property name="arm_radius" value="0.045" />
   <xacro:property name="arm_length" value="0.30" />
-  <xacro:property name="arm_mass" value="1.6" />
+  <xacro:property name="arm_mass" value="1.5" />
   <xacro:property name="arm_ixx" value="${(1.0/12.0) * arm_mass * (3 * arm_radius * arm_radius + arm_length * arm_length)}" />
   <xacro:property name="arm_iyy" value="${(1.0/12.0) * arm_mass * (3 * arm_radius * arm_radius + arm_length * arm_length)}" />
@@ -79,5 +79,5 @@
   <xacro:property name="forearm_radius" value="0.04" />
   <xacro:property name="forearm_length" value="0.26" />
-  <xacro:property name="forearm_mass" value="1.0" />
+  <xacro:property name="forearm_mass" value="0.9" />
   <xacro:property name="forearm_ixx" value="${(1.0/12.0) * forearm_mass * (3 * forearm_radius * forearm_radius + forearm_length * forearm_length)}" />
   <xacro:property name="forearm_iyy" value="${(1.0/12.0) * forearm_mass * (3 * forearm_radius * forearm_radius + forearm_length * forearm_length)}" />
@@ -87,5 +87,5 @@
   <xacro:property name="hand_width" value="0.09" />
   <xacro:property name="hand_height" value="0.03" />
-  <xacro:property name="hand_mass" value="0.6" />
+  <xacro:property name="hand_mass" value="0.5" />
   <xacro:property name="hand_ixx" value="${(1.0/12.0) * hand_mass * (hand_width * hand_width + hand_height * hand_height)}" />
   <xacro:property name="hand_iyy" value="${(1.0/12.0) * hand_mass * (hand_length * hand_length + hand_height * hand_height)}" />

Commit message: Update robot_stage5.xacro

File: robots/robot_stage5.xacro (robot description, xacro)
@@ -173,5 +173,5 @@
     <parent link="base_link"/>
     <child link="imu_link"/>
-    <origin xyz="${body_radius} 0 ${body_offset - body_length/4}" rpy="0 0 0"/>
+    <origin xyz="${body_radius + 0.05} 0 ${body_offset - body_length/4}" rpy="0 0 0"/>
   </joint>
   <!-- Neck -->

Commit message: retorno ao stabily pitch tentativa falhou

File: robots/robot_stage5.xacro (robot description, xacro)
@@ -173,5 +173,5 @@
     <parent link="base_link"/>
     <child link="imu_link"/>
-    <origin xyz="${body_radius + 0.05} 0 ${body_offset - body_length/4}" rpy="0 0 0"/>
+    <origin xyz="${body_radius + 0.1} 0 ${body_offset - body_length/4}" rpy="0 0 0"/>
   </joint>
   <!-- Neck -->

Commit message: ajuste

File: robots/robot_stage5.xacro (robot description, xacro)
@@ -393,5 +393,5 @@
       <origin xyz="0 0 ${-shin_length}"/>
       <axis xyz="0 1 0"/>
-      <limit lower="${-25 * deg_to_rad}" upper="${25 * deg_to_rad}" effort="${joint_effort}" velocity="${joint_velocity}"/>
+      <limit lower="${-20 * deg_to_rad}" upper="${20 * deg_to_rad}" effort="${joint_effort}" velocity="${joint_velocity}"/>
       <dynamics damping="${joint_damping}" friction="${joint_friction}"/>
     </joint>

Commit message: reversão no simple

File: robots/robot_stage5.xacro (robot description, xacro)
@@ -173,5 +173,5 @@
     <parent link="base_link"/>
     <child link="imu_link"/>
-    <origin xyz="${body_radius + 0.1} 0 ${body_offset - body_length/4}" rpy="0 0 0"/>
+    <origin xyz="${body_radius + 0.05} 0 ${body_offset - body_length/4}" rpy="0 0 0"/>
   </joint>
   <!-- Neck -->

Commit message: subiu a rampa

File: robots/robot_stage5.xacro (robot description, xacro)
@@ -393,5 +393,5 @@
       <origin xyz="0 0 ${-shin_length}"/>
       <axis xyz="0 1 0"/>
-      <limit lower="${-20 * deg_to_rad}" upper="${20 * deg_to_rad}" effort="${joint_effort}" velocity="${joint_velocity}"/>
+      <limit lower="${-25 * deg_to_rad}" upper="${25 * deg_to_rad}" effort="${joint_effort}" velocity="${joint_velocity}"/>
       <dynamics damping="${joint_damping}" friction="${joint_friction}"/>
     </joint>
