Commit message: ajuste no robo

File: robots/robot_stage5.xacro (robot description, xacro)
@@ -266,5 +266,5 @@
       <origin xyz="0 0 0"/>
       <axis xyz="1 0 0"/>
-      <limit lower="${-25 * deg_to_rad}" upper="${25 * deg_to_rad}" effort="${joint_effort}" velocity="${joint_velocity}"/>
+      <limit lower="${-15 * deg_to_rad}" upper="${15 * deg_to_rad}" effort="${joint_effort}" velocity="${joint_velocity}"/>
       <dynamics damping="${joint_damping}" friction="${joint_friction}"/>
     </joint>
@@ -422,5 +422,5 @@
       <origin xyz="0 0 0"/>
       <axis xyz="1 0 0"/>
-      <limit lower="${-15 * deg_to_rad}" upper="${15 * deg_to_rad}" effort="${joint_effort}" velocity="${joint_velocity}"/>
+      <limit lower="${-10 * deg_to_rad}" upper="${10 * deg_to_rad}" effort="${joint_effort}" velocity="${joint_velocity}"/>
       <dynamics damping="${joint_damping}" friction="${joint_friction}"/>
     </joint>

Commit message: alteração nas pernas e coxas

File: robots/robot_stage5.xacro (robot description, xacro)
@@ -30,5 +30,5 @@
   <!-- Thigh properties -->
   <xacro:property name="thigh_radius" value="0.075" />
-  <xacro:property name="thigh_length" value="0.40" />
+  <xacro:property name="thigh_length" value="0.43" />
   <xacro:property name="thigh_mass" value="16.0" />
   <xacro:property name="thigh_ixx" value="${(1.0/12.0) * thigh_mass * (3 * thigh_radius * thigh_radius + thigh_length * thigh_length)}" />
@@ -43,5 +43,5 @@
   <!-- Shin properties -->
   <xacro:property name="shin_radius" value="0.06" />
-  <xacro:property name="shin_length" value="0.43" />
+  <xacro:property name="shin_length" value="0.40" />
   <xacro:property name="shin_mass" value="7.3" />
   <xacro:property name="shin_ixx" value="${(1.0/12.0) * shin_mass * (3 * shin_radius * shin_radius + shin_length * shin_length)}" />
